File: CAM-XILINX_STM/com_1300/com_1300.kicad_pcb (KiCad board)
At the start: 6 copper layers, 50 x 66 mm, 129 parts, among them J1 Conn_02x20_Counter_Clockwise, J2 9-68RD-0.635SF, J3 MEC1-108-01-S-D-RA1-SL, J4 Conn_02x10_Top_Bottom, U1 LT1963AxST-3.3, U17 MT48LC16M16A2TG-7E, U2 STM32F415RGTx, U3 AM29LV320DT90EC, U4 TC74LCX373FT, U6 LP3982IMM-ADJ, U7 LTC3411EMS, Y1 16mHz, Y2 40mHZ

Commit message: test
Parts:
- R16: value R-OPEN -> 0
Connections:
- J2 pad 36: GND -> Net-(J2-CD1#)
- J2 pad 43: Net-(J2-Pad43) -> Net-(J2-CD1#)
- R16 pad 1: Net-(J2-Pad43) -> Net-(J2-CD1#)
Routing:
- net Net-(J2-Pad43): track 2.24 -> 0.00 mm, vias 1 -> 0
- net Net-(J2-CD1#): track 0.00 -> 2.24 mm, vias 0 -> 1
