File: CAM-XILINX_STM/com_1300/com_1300.kicad_sch (KiCad schematic)
At the start: 128 parts, among them J1 Conn_02x20_Counter_Clockwise, J2 9-68RD-0.635SF, J3 MEC1-108-01-S-D-RA1-SL, J4 Conn_02x10_Top_Bottom, U1 LT1963AxST-3.3, U17 MT48LC16M16A2TG-7E, U2 STM32F415RGTx, U3 AM29LV320DT90EC, U4 TC74LCX373FT, U6 LP3982IMM-ADJ, U7 LTC3411EMS, Y1 16mHz, Y2 40mHZ

Commit message: test
Parts:
- removed J1: Conn_02x20_Counter_Clockwise, Connector_PinSocket_2.00mm:PinSocket_2x20_P2.00mm_Horizontal, symbol Connector_Generic:Conn_02x20_Odd_Even
- R16: value R-OPEN -> 0
Connections:
- net GND: no longer J2.36 (CD1#)
- net at J2.43 (VS1#/Refresh), R16.1: now also J2.36 (CD1#)
- net USER_IO_0: no longer names the net of U.G2 (IO)
- net USER_IO_1: no longer names the net of U.C1 (IO_L01N_7/VRP_7)
- net USER_IO_10: no longer names the net of U.E2 (IO_L20P_7)
- net USER_IO_11: no longer names the net of U.F4 (IO_L21N_7)
- net USER_IO_12: no longer names the net of U.E4 (IO_L21P_7)
- net USER_IO_13: no longer names the net of U.F2 (IO_L22N_7)
- net USER_IO_14: no longer names the net of U.F3 (IO_L22P_7)
- net USER_IO_15: no longer names the net of U.G5 (IO_L23N_7)
- net USER_IO_16: no longer names the net of U.F5 (IO_L23P_7)
- net USER_IO_17: no longer names the net of U.G3 (IO_L24N_7)
- net USER_IO_18: no longer names the net of U.G4 (IO_L24P_7)
- net USER_IO_19: no longer names the net of U.H3 (IO_L39N_7)
- net USER_IO_2: no longer names the net of U.B1 (IO_L01P_7/VRN_7)
- net USER_IO_20: no longer names the net of U.H4 (IO_L39P_7)
- net USER_IO_21: no longer names the net of U.A9 (IO)
- net USER_IO_22: no longer names the net of U.A12 (IO)
- net USER_IO_23: no longer names the net of U.C10 (IO)
- net USER_IO_24: no longer names the net of U.D12 (IO/VREF_1)
- net USER_IO_25: no longer names the net of U.A14 (IO_L01N_1/VRP_1)
- net USER_IO_26: no longer names the net of U.B14 (IO_L01P_1/VRN_1)
- net USER_IO_27: no longer names the net of U.A13 (IO_L10N_1/VREF_1)
- net USER_IO_28: no longer names the net of U.B13 (IO_L10P_1)
- net USER_IO_29: no longer names the net of U.B12 (IO_L27N_1)
- net USER_IO_3: no longer names the net of U.C2 (IO_L16N_7)
- net USER_IO_30: no longer names the net of U.C12 (IO_L27P_1)
- net USER_IO_31: no longer names the net of U.D11 (IO_L28N_1)
- net USER_IO_4: no longer names the net of U.C3 (IO_L16P_7/VREF_7)
- net USER_IO_5: no longer names the net of U.D1 (IO_L17N_7)
- net USER_IO_6: no longer names the net of U.D2 (IO_L17P_7)
- net USER_IO_7: no longer names the net of U.E3 (IO_L19N_7/VREF_7)
- net USER_IO_8: no longer names the net of U.D3 (IO_L19P_7)
- net USER_IO_9: no longer names the net of U.E1 (IO_L20N_7)
- no-connect marks 14 -> 46
