File: CAM_XILINX_STM/com_1300/com_1300.kicad_pcb (KiCad board)
At the start: 6 copper layers, 50 x 66 mm, 129 parts, among them J1 Conn_02x20_Counter_Clockwise, J2 9-68RD-0.635SF, J3 MEC1-108-01-S-D-RA1-SL, J4 Conn_02x10_Top_Bottom, U1 LT1963AxST-3.3, U17 MT48LC16M16A2TG-7E, U2 STM32F415RGTx, U3 AM29LV320DT90EC, U4 TC74LCX373FT, U6 LP3982IMM-ADJ, U7 LTC3411EMS, Y1 16mHz, Y2 40mHZ

Commit message: 22323
Parts:
- removed the C24 at (40.2, 40.4)
- removed the C24 at (16.1, 40.5)
- removed the C24 at (53.9, 27.0)
- removed the C24 at (51.2, 41.5)
- removed the C24 at (63.8, 40.4)
- removed the C24 at (63.8, 34.3)
- removed the C24 at (63.8, 28.2)
- removed the C24 at (40.2, 28.2)
- removed the C24 at (45.9, 27.1)
- removed R17: R-OPEN, Resistor_SMD:R_0402_1005Metric
- removed RN8: 8 x 10K, Resistor_SMD:R_Cat16-8
- removed U17: MT48LC16M16A2TG-7E, Package_SO:TSOP-II-54_22.2x10.16mm_P0.8mm
- R16: value R-OPEN -> 0
Connections:
- net INOUT_PC_CARD_14 renamed INOUT_WE#
- net INOUT_PC_CARD_15 renamed INOUT_MIVAL
- net INOUT_PC_CARD_16 renamed INOUT_MCLKI
- net INOUT_PC_CARD_18 renamed INOUT_A7
- net INOUT_PC_CARD_19 renamed INOUT_A6
- net INOUT_PC_CARD_20 renamed INOUT_A5
- net INOUT_PC_CARD_21 renamed INOUT_A4
- net INOUT_PC_CARD_22 renamed INOUT_A3
- net INOUT_PC_CARD_23 renamed INOUT_A2
- net INOUT_PC_CARD_24 renamed INOUT_A1
- net INOUT_PC_CARD_25 renamed INOUT_A0
- net INOUT_PC_CARD_26 renamed INOUT_D0
- net INOUT_PC_CARD_27 renamed INOUT_D1
- net INOUT_PC_CARD_30 renamed INOUT_MDO3
- net INOUT_PC_CARD_31 renamed INOUT_MDO4
- net INOUT_PC_CARD_32 renamed INOUT_MDO5
- net INOUT_PC_CARD_33 renamed INOUT_MDO6
- net INOUT_PC_CARD_34 renamed INOUT_MDO7
- net INOUT_PC_CARD_36 renamed INOUT_IORD#
- net INOUT_PC_CARD_37 renamed INOUT_IOWR#
- net INOUT_PC_CARD_38 renamed INOUT_MISTRT
- net INOUT_PC_CARD_39 renamed INOUT_MDI0
- net INOUT_PC_CARD_40 renamed INOUT_MDI1
- net INOUT_PC_CARD_41 renamed INOUT_MDI2
- net INOUT_PC_CARD_42 renamed INOUT_MDI3
- net INOUT_PC_CARD_43 renamed INOUT_MDI4
- net INOUT_PC_CARD_44 renamed INOUT_MDI5
- net INOUT_PC_CARD_45 renamed INOUT_MDI6
- net INOUT_PC_CARD_46 renamed INOUT_MDI7
- net INOUT_PC_CARD_48 renamed INOUT_INPACK#
- net INOUT_PC_CARD_49 renamed INOUT_REG#
- net INOUT_PC_CARD_50 renamed INOUT_MOVAL
- net INOUT_PC_CARD_51 renamed INOUT_MOSTRT
- net INOUT_PC_CARD_52 renamed INOUT_MDO0
- net INOUT_PC_CARD_53 renamed INOUT_MDO1
- net INOUT_PC_CARD_54 renamed INOUT_MDO2
- net INOUT_PC_CARD_6 renamed INOUT_CE1#
- net INOUT_PC_CARD_8 renamed INOUT_OE#
- net INOUT_PC_CARD_RESET renamed INOUT_RESET
- net PC_CARD_1 renamed D3
- net PC_CARD_14 renamed WE#
- net PC_CARD_15 renamed MIVAL
- net PC_CARD_16 renamed MCLKI
- net PC_CARD_18 renamed A7
- net PC_CARD_19 renamed A6
- net PC_CARD_2 renamed D4
- net PC_CARD_20 renamed A5
- net PC_CARD_21 renamed A4
- net PC_CARD_22 renamed A3
- net PC_CARD_23 renamed A2
- net PC_CARD_24 renamed A1
- net PC_CARD_25 renamed A0
- net PC_CARD_26 renamed D0
- net PC_CARD_27 renamed D1
- net PC_CARD_28 renamed D2
- net PC_CARD_3 renamed D5
- net PC_CARD_30 renamed MDO3
- net PC_CARD_31 renamed MDO4
- net PC_CARD_32 renamed MDO5
- net PC_CARD_33 renamed MDO6
- net PC_CARD_34 renamed MDO7
- net PC_CARD_36 renamed IORD#
- net PC_CARD_37 renamed IOWR#
- net PC_CARD_38 renamed MISTRT
- net PC_CARD_39 renamed MDI0
- net PC_CARD_4 renamed D6
- net PC_CARD_40 renamed MDI1
- net PC_CARD_41 renamed MDI2
- net PC_CARD_42 renamed MDI3
- net PC_CARD_43 renamed MDI4
- net PC_CARD_44 renamed MDI5
- net PC_CARD_45 renamed MDI6
- net PC_CARD_46 renamed MDI7
- net PC_CARD_48 renamed INPACK#
- net PC_CARD_49 renamed REG#
- net PC_CARD_5 renamed D7
- net PC_CARD_50 renamed MOVAL
- net PC_CARD_51 renamed MOSTRT
- net PC_CARD_52 renamed MDO0
- net PC_CARD_53 renamed MDO1
- net PC_CARD_54 renamed MDO2
- net PC_CARD_55 renamed IREQ#
- net PC_CARD_6 renamed CE1#
- net PC_CARD_8 renamed OE#
- net PC_CARD_RESET renamed RESET
- C27 pad 1: FPGA_CLK1 -> /FPGA_CLK1
- J2 pad 10: PC_CARD_9 -> unconnected-(J2-A11-Pad10)
- J2 pad 11: PC_CARD_10 -> unconnected-(J2-A9-Pad11)
- J2 pad 12: PC_CARD_11 -> unconnected-(J2-A8-Pad12)
- J2 pad 13: PC_CARD_12 -> unconnected-(J2-A13-Pad13)
- J2 pad 14: PC_CARD_13 -> unconnected-(J2-A14-Pad14)
- J2 pad 18: unconnected-(J2-Pad18) -> VCC
- J2 pad 21: PC_CARD_17 -> unconnected-(J2-A12-Pad21)
- J2 pad 33: PC_CARD_29 -> unconnected-(J2-IOIS16#-Pad33)
- J2 pad 36: Net-(J2-Pad36) -> Net-(J2-CD1#)
- J2 pad 42: PC_CARD_35 -> unconnected-(J2-CE2#-Pad42)
- J2 pad 43: Net-(J2-Pad36) -> unconnected-(J2-VS1#/Refresh-Pad43)
- J2 pad 52: unconnected-(J2-Pad52) -> VCC
- J2 pad 57: Net-(J2-Pad57) -> MCLKO
- J2 pad 59: PC_CARD_47 -> unconnected-(J2-WAIT#-Pad59)
- J2 pad 8: PC_CARD_7 -> unconnected-(J2-A10-Pad8)
- J4 pad 1: TIM3_CH4 -> unconnected-(J4-Pin_1-Pad1)
- J4 pad 10: SPI2_MOSI -> unconnected-(J4-Pin_10-Pad10)
- J4 pad 11: GPIO_1 -> unconnected-(J4-Pin_11-Pad11)
- J4 pad 12: USB_D- -> unconnected-(J4-Pin_12-Pad12)
- J4 pad 13: SWCLK -> unconnected-(J4-Pin_13-Pad13)
- J4 pad 14: USB_D+ -> unconnected-(J4-Pin_14-Pad14)
- J4 pad 2: USART3_RX -> unconnected-(J4-Pin_2-Pad2)
- J4 pad 3: TIM3_CH3 -> unconnected-(J4-Pin_3-Pad3)
- J4 pad 4: USART3_CK -> unconnected-(J4-Pin_4-Pad4)
- J4 pad 5: CAN2_RX -> unconnected-(J4-Pin_5-Pad5)
- J4 pad 6: SPI2_SCK -> unconnected-(J4-Pin_6-Pad6)
- J4 pad 7: CAN2_TX -> unconnected-(J4-Pin_7-Pad7)
- J4 pad 8: SPI2_MISO -> unconnected-(J4-Pin_8-Pad8)
- J4 pad 9: USART3_TX -> unconnected-(J4-Pin_9-Pad9)
- R10 pad 2: FPGA_CLK1 -> /FPGA_CLK1
- R16 pad 1: Net-(J2-Pad36) -> Net-(J2-CD1#)
- R3 pad 1: BOOT0 -> unconnected-(R3-Pad1)
- R9 pad 2: SWIDO -> unconnected-(R9-Pad2)
- RN1 pad 6: INOUT_PC_CARD_28 -> INOUT_D2
- RN1 pad 8: INOUT_PC_CARD_29 -> unconnected-(RN1-R8.1-Pad8)
- RN1 pad 9: PC_CARD_29 -> unconnected-(RN1-R8.2-Pad9)
- RN2 pad 1: INOUT_PC_CARD_47 -> unconnected-(RN2-R1.1-Pad1)
- RN2 pad 16: PC_CARD_47 -> unconnected-(RN2-R1.2-Pad16)
- RN3 pad 1: INOUT_PC_CARD_17 -> unconnected-(RN3-R1.1-Pad1)
- RN3 pad 16: PC_CARD_17 -> unconnected-(RN3-R1.2-Pad16)
- RN4 pad 3: INOUT_PC_CARD_55 -> INOUT_IREQ#
- RN5 pad 1: INOUT_PC_CARD_10 -> unconnected-(RN5-R1.1-Pad1)
- RN5 pad 10: PC_CARD_13 -> unconnected-(RN5-R7.2-Pad10)
- RN5 pad 12: PC_CARD_12 -> unconnected-(RN5-R5.2-Pad12)
- RN5 pad 14: PC_CARD_11 -> unconnected-(RN5-R3.2-Pad14)
- RN5 pad 16: PC_CARD_10 -> unconnected-(RN5-R1.2-Pad16)
- RN5 pad 3: INOUT_PC_CARD_11 -> unconnected-(RN5-R3.1-Pad3)
- RN5 pad 5: INOUT_PC_CARD_12 -> unconnected-(RN5-R5.1-Pad5)
- RN5 pad 7: INOUT_PC_CARD_13 -> unconnected-(RN5-R7.1-Pad7)
- RN6 pad 10: PC_CARD_9 -> unconnected-(RN6-R7.2-Pad10)
- RN6 pad 12: PC_CARD_35 -> unconnected-(RN6-R5.2-Pad12)
- RN6 pad 13: PC_CARD_7 -> MCLKO
- RN6 pad 4: INOUT_PC_CARD_7 -> INOUT_MCLKO
- RN6 pad 5: INOUT_PC_CARD_35 -> unconnected-(RN6-R5.1-Pad5)
- RN6 pad 7: INOUT_PC_CARD_9 -> unconnected-(RN6-R7.1-Pad7)
- RN7 pad 1: INOUT_PC_CARD_1 -> INOUT_D3
- RN7 pad 2: INOUT_PC_CARD_2 -> INOUT_D2
- RN7 pad 4: INOUT_PC_CARD_3 -> INOUT_D5
- RN7 pad 6: INOUT_PC_CARD_4 -> INOUT_D6
- RN7 pad 8: INOUT_PC_CARD_5 -> INOUT_D7
- U pad A12: USER_IO_22 -> unconnected-(U5-IO-PadA12)
- U pad A13: USER_IO_27 -> unconnected-(U5-IO_L10N_1/VREF_1-PadA13)
- U pad A14: USER_IO_25 -> unconnected-(U5-IO_L01N_1/VRP_1-PadA14)
- U pad A4: SERIAL_IO_1 -> unconnected-(U5-IO_L01P_0/VRN_0-PadA4)
- U pad A9: USER_IO_21 -> unconnected-(U5-IO-PadA9)
- U pad B1: USER_IO_2 -> unconnected-(U5-IO_L01P_7/VRN_7-PadB1)
- U pad B12: USER_IO_29 -> unconnected-(U5-IO_L27N_1-PadB12)
- U pad B13: USER_IO_28 -> unconnected-(U5-IO_L10P_1-PadB13)
- U pad B14: USER_IO_26 -> unconnected-(U5-IO_L01P_1/VRN_1-PadB14)
- U pad B8: unconnected-(U5-PadB8) -> INOUT_MCLKO
- U pad C1: USER_IO_1 -> unconnected-(U5-IO_L01N_7/VRP_7-PadC1)
- U pad C10: USER_IO_23 -> unconnected-(U5-IO-PadC10)
- U pad C12: USER_IO_30 -> unconnected-(U5-IO_L27P_1-PadC12)
- U pad C15: SDRAM_A1 -> unconnected-(U5-IO_L16N_2-PadC15)
- U pad C16: SDRAM_A0 -> unconnected-(U5-IO_L01P_2/VRN_2-PadC16)
- U pad C2: USER_IO_3 -> unconnected-(U5-IO_L16N_7-PadC2)
- U pad C3: USER_IO_4 -> unconnected-(U5-IO_L16P_7/VREF_7-PadC3)
- U pad C5: SERIAL_IO_2 -> unconnected-(U5-IO_L25N_0-PadC5)
- U pad D1: USER_IO_5 -> unconnected-(U5-IO_L17N_7-PadD1)
- U pad D11: USER_IO_31 -> unconnected-(U5-IO_L28N_1-PadD11)
- U pad D12: USER_IO_24 -> unconnected-(U5-IO/VREF_1-PadD12)
- U pad D14: SDRAM_A2 -> unconnected-(U5-IO_L16P_2-PadD14)
- U pad D15: SDRAM_A3 -> unconnected-(U5-IO_L17N_2-PadD15)
- U pad D16: SDRAM_A4 -> unconnected-(U5-IO_L17P_2/VREF_2-PadD16)
- U pad D2: USER_IO_6 -> unconnected-(U5-IO_L17P_7-PadD2)
- U pad D3: USER_IO_8 -> unconnected-(U5-IO_L19P_7-PadD3)
- U pad D5: FPGA_CLK1 -> unconnected-(U5-IO_VREF_0-PadD5)
- U pad E1: USER_IO_9 -> unconnected-(U5-IO_L20N_7-PadE1)
- U pad E13: SDRAM_A5 -> unconnected-(U5-IO_L19N_2-PadE13)
- U pad E14: SDRAM_A6 -> unconnected-(U5-IO_L19P_2-PadE14)
- U pad E15: SDRAM_A7 -> unconnected-(U5-IO_L20N_2-PadE15)
- U pad E16: SDRAM_A8 -> unconnected-(U5-IO_L20P_2-PadE16)
- U pad E2: USER_IO_10 -> unconnected-(U5-IO_L20P_7-PadE2)
- U pad E3: USER_IO_7 -> unconnected-(U5-IO_L19N_7/VREF_7-PadE3)
- U pad E4: USER_IO_12 -> unconnected-(U5-IO_L21P_7-PadE4)
- U pad F12: SDRAM_A9 -> unconnected-(U5-IO_L21N_2-PadF12)
- U pad F13: SDRAM_A10 -> unconnected-(U5-IO_L21P_2-PadF13)
- U pad F14: SDRAM_A11 -> unconnected-(U5-IO_L22N_2-PadF14)
- U pad F15: SDRAM_A12 -> unconnected-(U5-IO_L22P_2-PadF15)
- U pad F2: USER_IO_13 -> unconnected-(U5-IO_L22N_7-PadF2)
- U pad F3: USER_IO_14 -> unconnected-(U5-IO_L22P_7-PadF3)
- U pad F4: USER_IO_11 -> unconnected-(U5-IO_L21N_7-PadF4)
- U pad F5: USER_IO_16 -> unconnected-(U5-IO_L23P_7-PadF5)
- U pad G1: INOUT_PC_CARD_55 -> INOUT_IREQ#
- U pad G12: SDRAM_DQ0 -> unconnected-(U5-IO_L23N_2/VREF_2-PadG12)
- U pad G13: SDRAM_DQ1 -> unconnected-(U5-IO_L23P_2-PadG13)
- U pad G14: SDRAM_DQ2 -> unconnected-(U5-IO_L24N_2-PadG14)
- U pad G15: SDRAM_DQ3 -> unconnected-(U5-IO_L24P_2-PadG15)
- U pad G2: USER_IO_0 -> unconnected-(U5-IO-PadG2)
- U pad G3: USER_IO_17 -> unconnected-(U5-IO_L24N_7-PadG3)
- U pad G4: USER_IO_18 -> unconnected-(U5-IO_L24P_7-PadG4)
- U pad G5: USER_IO_15 -> unconnected-(U5-IO_L23N_7-PadG5)
- U pad H13: SDRAM_DQ4 -> unconnected-(U5-IO_L39N_2-PadH13)
- U pad H14: SDRAM_DQ5 -> unconnected-(U5-IO_L39P_2-PadH14)
- U pad H15: SDRAM_DQ6 -> unconnected-(U5-IO_L40N_2-PadH15)
- U pad H16: SDRAM_DQ7 -> unconnected-(U5-IO_L40P_2/VREF_2-PadH16)
- U pad H3: USER_IO_19 -> unconnected-(U5-IO_L39N_7-PadH3)
- U pad H4: USER_IO_20 -> unconnected-(U5-IO_L39P_7-PadH4)
- U pad J13: INOUT_PC_CARD_3 -> unconnected-(U5-IO_L39P_3-PadJ13)
- U pad J14: INOUT_PC_CARD_2 -> unconnected-(U5-IO_L39N_3-PadJ14)
- U pad J16: INOUT_PC_CARD_4 -> unconnected-(U5-IO_L40N_3/VREF_3-PadJ16)
- U pad J4: INOUT_PC_CARD_35 -> unconnected-(U5-IO_L39N_6-PadJ4)
- U pad K12: SDRAM_CNTRL3 -> unconnected-(U5-IO_L23N_3-PadK12)
- U pad K13: INOUT_PC_CARD_1 -> unconnected-(U5-IO_L24P_3-PadK13)
- U pad K14: SDRAM_CNTRL1 -> unconnected-(U5-IO_L24N_3-PadK14)
- U pad K15: SDRAM_DQ8 -> unconnected-(U5-IO-PadK15)
- U pad K16: INOUT_PC_CARD_5 -> unconnected-(U5-IO_L40P_3-PadK16)
- U pad L12: SDRAM_CNTRL2 -> unconnected-(U5-IO_L23P_3/VREF_3-PadL12)
- U pad L13: SDRAM_CNTRL7 -> unconnected-(U5-IO_L21N_3-PadL13)
- U pad L14: SDRAM_CNTRL4 -> unconnected-(U5-IO_L22P_3-PadL14)
- U pad L15: SDRAM_CNTRL5 -> unconnected-(U5-IO_L22N_3-PadL15)
- U pad M13: SDRAM_CNTRL6 -> unconnected-(U5-IO_L21P_3-PadM13)
- U pad M14: SDRAM_DQ15 -> unconnected-(U5-IO_L19N_3-PadM14)
- U pad M15: SDRAM_CNTRL8 -> unconnected-(U5-IO_L20P_3-PadM15)
- U pad M16: SDRAM_CNTRL9 -> unconnected-(U5-IO_L20N_3-PadM16)
- U pad M4: INOUT_PC_CARD_47 -> unconnected-(U5-IO_L19N_6-PadM4)
- U pad N14: SDRAM_CNTRL10 -> unconnected-(U5-IO_L19P_3-PadN14)
- U pad N15: SDRAM_DQ14 -> unconnected-(U5-IO_L17P_3/VREF_3-PadN15)
- U pad N16: SDRAM_DQ13 -> unconnected-(U5-IO_L17N_3-PadN16)
- U pad P12: INOUT_PC_CARD_13 -> unconnected-(U5-IO_L25N_4-PadP12)
- U pad P13: INOUT_PC_CARD_9 -> unconnected-(U5-IO/VREF_4-PadP13)
- U pad P14: SDRAM_DQ12 -> unconnected-(U5-IO_L16P_3-PadP14)
- U pad P15: SDRAM_DQ11 -> unconnected-(U5-IO_L16N_3-PadP15)
- U pad P16: SDRAM_DQ9 -> unconnected-(U5-IO_L01N_3/VRP_3-PadP16)
- U pad R11: INOUT_PC_CARD_17 -> unconnected-(U5-IO_L28P_4-PadR11)
- U pad R13: INOUT_PC_CARD_11 -> unconnected-(U5-IO_L01N_4/VRP_4-PadR13)
- U pad R16: SDRAM_DQ10 -> unconnected-(U5-IO_L01P_3/VRN_3-PadR16)
- U pad T10: INOUT_PC_CARD_10 -> unconnected-(U5-IO/VREF_4-PadT10)
- U pad T13: INOUT_PC_CARD_12 -> unconnected-(U5-IO_L01P_4/VRN_4-PadT13)
- U pad T14: INOUT_PC_CARD_7 -> unconnected-(U5-IO-PadT14)
- U pad T5: INOUT_PC_CARD_29 -> unconnected-(U5-IO-PadT5)
- U pad T8: INOUT_PC_CARD_28 -> INOUT_D2
- U2 pad 15: BOOT_SECTOR -> unconnected-(U2-PA1-Pad15)
- U2 pad 26: TIM3_CH3 -> unconnected-(U2-PB0-Pad26)
- U2 pad 27: TIM3_CH4 -> unconnected-(U2-PB1-Pad27)
- U2 pad 30: USART3_RX -> unconnected-(U2-PB11-Pad30)
- U2 pad 33: USART3_CK -> unconnected-(U2-PB12-Pad33)
- U2 pad 34: SPI2_SCK -> unconnected-(U2-PB13-Pad34)
- U2 pad 35: SPI2_MISO -> unconnected-(U2-PB14-Pad35)
- U2 pad 36: SPI2_MOSI -> unconnected-(U2-PB15-Pad36)
- U2 pad 44: USB_D- -> unconnected-(U2-PA11-Pad44)
- U2 pad 45: USB_D+ -> unconnected-(U2-PA12-Pad45)
- U2 pad 46: SWIDO -> unconnected-(U2-PA13-Pad46)
- U2 pad 49: SWCLK -> unconnected-(U2-PA14-Pad49)
- U2 pad 50: GPIO_1 -> unconnected-(U2-PA15-Pad50)
- U2 pad 51: USART3_TX -> unconnected-(U2-PC10-Pad51)
- U2 pad 58: CAN2_TX -> unconnected-(U2-PB6-Pad58)
- U2 pad 59: CAN2_RX -> unconnected-(U2-PB7-Pad59)
- U2 pad 60: BOOT0 -> unconnected-(U2-BOOT0-Pad60)
Routing:
- net (no net): track 0.00 -> 1131.5 mm, vias 0 -> 62
- net INOUT_PC_CARD_35: track 73.4 -> 0.00 mm, vias 3 -> 0
- net INOUT_PC_CARD_3: track 65.4 -> 0.00 mm, vias 3 -> 0
- net INOUT_PC_CARD_2: track 64.5 -> 0.00 mm, vias 3 -> 0
- net INOUT_PC_CARD_5: track 61.1 -> 0.00 mm, vias 3 -> 0
- net INOUT_PC_CARD_1: track 56.1 -> 0.00 mm, vias 3 -> 0
- net INOUT_PC_CARD_47: track 48.7 -> 0.00 mm, vias 3 -> 0
- net INOUT_PC_CARD_13: track 48.5 -> 0.00 mm, vias 2 -> 0
- net INOUT_PC_CARD_4: track 48.0 -> 0.00 mm, vias 3 -> 0
- net INOUT_PC_CARD_9: track 47.7 -> 0.00 mm, vias 3 -> 0
- net INOUT_PC_CARD_10: track 46.9 -> 0.00 mm, vias 4 -> 0
- net INOUT_PC_CARD_11: track 46.6 -> 0.00 mm, vias 2 -> 0
- net INOUT_PC_CARD_12: track 45.8 -> 0.00 mm, vias 2 -> 0
- net INOUT_PC_CARD_7: track 45.4 -> 0.00 mm, vias 2 -> 0
- net SDRAM_A2: track 44.8 -> 0.00 mm, vias 3 -> 0
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
Commit message: 124214
Parts:
- removed the J1 at (59.0, 25.0) (x2)
- removed J4: Conn_02x10_Top_Bottom, Connector_PinHeader_1.27mm:PinHeader_2x08_P1.27mm_Vertical_SMD
- removed the R3 at (35.0, 51.4)
- removed the R9 at (38.0, 51.6)
- C24: moved to F.Cu
- R15: renamed from R16; moved to F.Cu
- R16: renamed from R15; moved to F.Cu
- R5: renamed from R11; moved to F.Cu
- moved C58 57.6 mm to (30.7, 11.4)
- moved U2 50.3 mm to (21.3, 19.8)
- moved C53 48.9 mm to (45.2, 19.1)
- moved R16 46.5 mm to (30.2, 34.3)
- moved J1 45.1 mm to (22.5, 10.2)
- moved U3 44.5 mm to (50.5, 32.3)
- moved L1 42.9 mm to (59.2, 48.0), turned to 180 degrees
- moved U7 42.4 mm to (37.8, 10.4), turned to -90 degrees
- moved C24 41.0 mm to (49.1, 39.3), turned to 90 degrees
- moved C24 39.9 mm to (49.1, 36.5), turned to 90 degrees
- moved U6 38.5 mm to (55.6, 18.0), turned to -90 degrees
- moved R17 38.5 mm to (55.2, 48.5)
- moved C24 38.5 mm to (46.5, 30.2)
- moved Y1 38.3 mm to (45.8, 27.0)
- moved C24 38.2 mm to (50.8, 36.7)
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- renumbered C16 to C33, C25 to C35, C23 to C36, C22 to C37, C4 to C39, C9 to C49, C12 to C50, C8 to C51, C18 to C52, C2 to C53, C19 to C54, C1 to C55, C20 to C56, C10 to C57, C17 to C58, C15 to C59, C14 to C60, C27 to C61, C26 to C62, J3 to J1, R12 to R1, R5 to R10, R7 to R11, R23 to R12, R10 to R13, R6 to R14, R1 to R17, R4 to R2, R2 to R3, R14 to R4, R13 to R6, R8 to R7, R21 to R9, RN3 to RN2, RN5 to RN3, RN7 to RN4, RN2 to RN5, RN4 to RN6, RN6 to RN7, U6 to U2, U7 to U3, U2 to U5, U3 to U6, U4 to U7, Y2 to Y1, Y1 to Y2
Routing:
- net (no net): track 1131.5 -> 0.00 mm, vias 62 -> 0
- net GND: track 296.0 -> 144.3 mm, vias 68 -> 50
- net Net-(C40-Pad1): track 4.28 -> 119.7 mm, vias 0 -> 2
- net FPGA_CLK1: track 101.3 -> 0.00 mm, vias 3 -> 0
- net +3V3: track 121.6 -> 26.8 mm, vias 50 -> 1
- net uC_CNTRL2: track 107.2 -> 18.4 mm, vias 6 -> 1
- net INOUT_MDO5: track 85.7 -> 0.00 mm, vias 2 -> 0
- net FPGA_TEST_EDGE2: track 84.5 -> 0.00 mm, vias 3 -> 0
- net INOUT_MDO6: track 83.7 -> 0.00 mm, vias 2 -> 0
- net uC_AD6: track 83.6 -> 0.00 mm, vias 4 -> 0
- net INOUT_MDO7: track 83.5 -> 0.00 mm, vias 3 -> 0
- net INOUT_PC_CARD_55: track 80.8 -> 0.00 mm, vias 4 -> 0
- net INOUT_IORD#: track 75.9 -> 0.00 mm, vias 2 -> 0
- net VCC: track 82.8 -> 8.26 mm, vias 3 -> 0
- net USER_IO_0: track 72.7 -> 0.00 mm
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- removed copper zone on In1.Cu, net +2V5
- removed copper zone on In4.Cu, net +3V3
- removed copper zone on F.Cu, net GND
- removed copper zone on In3.Cu, net GND
- removed copper zone on In3.Cu, net uC_AD6
Other:
- board size 50 x 66 mm -> 50 x 75.9 mm
- copper layers 6 -> 4
