File: CAM_XILINX_STM/com_1300/com_1300.kicad_pcb (KiCad board)
At the start: 4 copper layers, 50 x 75.9 mm, 112 parts, among them J1 MEC1-108-01-S-D-RA1-SL, J2 9-68RD-0.635SF, U1 LT1963AxST-3.3, U2 LP3982IMM-ADJ, U3 LTC3411EMS, U5 STM32F415RGTx, U6 AM29LV320DT90EC, U7 TC74LCX373FT, Y1 40mHZ, Y2 16mHz

Commit message: 234
Parts:
- moved C24 7.48 mm to (37.3, 49.0)
- moved C24 7.48 mm to (39.1, 46.5)
- moved C24 7.48 mm to (39.1, 45.8)
- moved C24 7.48 mm to (28.5, 37.5)
- moved C24 7.48 mm to (43.5, 53.0)
- moved C24 7.48 mm to (39.1, 45.1)
- moved C24 7.48 mm to (39.1, 47.2)
- moved C24 7.48 mm to (39.1, 50.8)
- moved C24 7.48 mm to (43.0, 49.0)
- moved C24 7.48 mm to (35.2, 49.0)
- moved C24 7.48 mm to (42.3, 49.0)
- moved C24 7.48 mm to (35.5, 53.0)
- moved C24 7.48 mm to (39.1, 52.2)
- moved C24 7.48 mm to (39.1, 47.9)
- moved C24 7.48 mm to (39.1, 52.9)
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Routing:
- net VCC: track 8.12 -> 86.4 mm, vias 0 -> 2
- net FPGA_CNTRL3: track 0.00 -> 70.4 mm, vias 0 -> 5
- net uC_A14: track 0.00 -> 66.8 mm, vias 0 -> 2
- net uC_CNTRL2: track 18.3 -> 69.4 mm, vias 1 -> 3
- net +2V5: track 75.6 -> 120.1 mm, vias 0 -> 3
- net /FPGA_CLK1: track 0.00 -> 43.9 mm, vias 0 -> 2
- net INOUT_CE1#: track 0.00 -> 26.3 mm
- net FPGA_TEST_EDGE4: track 0.00 -> 3.83 mm
- net GND: track 149.1 -> 145.2 mm

Commit message: 2342342
Parts:
- removed the C24 at (32.4, 39.0)
- removed the C24 at (50.8, 36.7)
- removed the C24 at (50.8, 39.0)
- removed the C24 at (63.2, 55.6)
- removed the C24 at (21.2, 51.8)
- removed the C24 at (17.8, 33.2)
- removed the C24 at (41.7, 46.6)
- removed the C24 at (49.1, 39.3)
- removed the C24 at (21.7, 46.5)
- removed the C24 at (53.6, 59.8)
- removed the C24 at (51.1, 46.8)
- removed the C24 at (50.0, 46.9)
- removed the C24 at (49.1, 36.5)
- removed the C24 at (41.8, 51.4)
- removed the C24 at (17.8, 35.1)
- removed the C24 at (39.1, 46.5)
- removed the C24 at (39.1, 45.8)
- removed the C24 at (36.0, 45.0)
- removed the C24 at (28.5, 37.5)
- removed the C24 at (43.5, 53.0)
- removed the C24 at (39.1, 45.1)
- removed the C24 at (40.2, 49.0)
- removed the C24 at (46.5, 30.2)
- removed the C24 at (43.7, 49.0)
- removed the C24 at (39.1, 47.2)
- removed the C24 at (39.1, 50.8)
- removed the C24 at (43.0, 49.0)
- removed the C24 at (35.2, 49.0)
- removed the C24 at (42.3, 49.0)
- removed the C24 at (35.5, 53.0)
- removed the C24 at (39.1, 52.2)
- removed the C24 at (38.0, 49.0)
- removed the C24 at (34.5, 49.0)
- removed the C24 at (53.4, 45.0)
- removed the C24 at (34.8, 45.0)
- removed the C24 at (39.1, 47.9)
- removed the C24 at (39.1, 52.9)
- removed the C24 at (39.5, 49.0)
- removed the C24 at (40.9, 49.0)
- removed the C24 at (39.1, 51.5)
- removed the C24 at (36.6, 49.0)
- removed the C24 at (42.8, 45.0)
- removed the C24 at (41.6, 49.0)
- removed the C24 at (37.3, 49.0)
- removed the C24 at (29.2, 39.0)
- removed the C24 at (35.9, 49.0)
- removed the C24 at (42.8, 53.0)
- removed the C24 at (34.8, 53.0)
- removed the C24 at (35.5, 45.0)
- removed the C24 at (39.1, 50.1)
- removed the C24 at (38.8, 49.0)
- removed the C24 at (51.7, 51.3)
- removed the C24 at (44.9, 59.7)
- removed the C24 at (53.1, 43.6)
- removed the C24 at (37.3, 33.8)
- removed C39: 10uF, Capacitor_Tantalum_SMD:CP_EIA-3216-18_Kemet-A
- removed C62: C-OPEN, Capacitor_SMD:C_0402_1005Metric
- removed R9: 56, Resistor_SMD:R_0402_1005Metric
- removed U: XC3S400-4FT256C, Package_BGA:Xilinx_FTG256
- removed U7: TC74LCX373FT, Package_SO:SSOP-20_4.4x6.5mm_P0.65mm
- added C24: C-OPEN, Capacitor_SMD:C_0402_1005Metric, F.Cu at (41.5, 66.2)
- added C24: C-OPEN, Capacitor_SMD:C_0201_0603Metric, F.Cu at (38.3, 61.2)
- added C24: C-OPEN, Capacitor_SMD:C_0201_0603Metric, F.Cu at (35.8, 52.4)
- added C24: C-OPEN, Capacitor_SMD:C_0201_0603Metric, F.Cu at (38.3, 54.2)
- added C24: C-OPEN, Capacitor_SMD:C_0201_0603Metric, F.Cu at (39.4, 45.7)
- added C24: C-OPEN, Capacitor_SMD:C_0201_0603Metric, F.Cu at (40.7, 61.2)
- added C24: C-OPEN, Capacitor_SMD:C_0201_0603Metric, F.Cu at (35.8, 57.7)
- added C24: C-OPEN, Capacitor_SMD:C_0402_1005Metric, F.Cu at (37.6, 71.4)
- added C24: C-OPEN, Capacitor_SMD:C_0201_0603Metric, F.Cu at (36.9, 38.7)
- added C24: C-OPEN, Capacitor_SMD:C_0201_0603Metric, F.Cu at (38.3, 52.4)
- added C24: C-OPEN, Capacitor_SMD:C_0201_0603Metric, F.Cu at (35.8, 61.2)
- added C24: C-OPEN, Capacitor_SMD:C_0201_0603Metric, F.Cu at (34.5, 38.7)
- added C24: C-OPEN, Capacitor_SMD:C_0201_0603Metric, F.Cu at (40.7, 50.7)
- added C24: C-OPEN, Capacitor_SMD:C_0201_0603Metric, F.Cu at (43.2, 55.9)
- added C24: C-OPEN, Capacitor_SMD:C_0201_0603Metric, F.Cu at (36.9, 43.7)
- added C24: C-OPEN, Capacitor_SMD:C_0201_0603Metric, F.Cu at (34.5, 40.6)
- added C24: C-OPEN, Capacitor_SMD:C_0201_0603Metric, F.Cu at (36.9, 41.7)
- added C24: C-OPEN, Capacitor_SMD:C_0201_0603Metric, F.Cu at (40.7, 57.7)
- added C24: C-OPEN, Capacitor_SMD:C_0201_0603Metric, F.Cu at (38.3, 57.7)
- added C24: C-OPEN, Capacitor_SMD:C_0201_0603Metric, F.Cu at (38.3, 59.4)
- added C24: C-OPEN, Capacitor_SMD:C_0201_0603Metric, F.Cu at (34.5, 39.6)
- added C24: C-OPEN, Capacitor_SMD:C_0201_0603Metric, F.Cu at (36.9, 42.7)
- added C24: C-OPEN, Capacitor_SMD:C_0201_0603Metric, F.Cu at (34.5, 43.7)
- added C24: C-OPEN, Capacitor_SMD:C_0402_1005Metric, F.Cu at (34.8, 68.3)
- added C24: C-OPEN, Capacitor_SMD:C_0201_0603Metric, F.Cu at (39.3, 42.7)
- added C24: C-OPEN, Capacitor_SMD:C_0201_0603Metric, F.Cu at (35.8, 55.9)
- added C24: C-OPEN, Capacitor_SMD:C_0201_0603Metric, F.Cu at (35.8, 54.2)
- added C24: C-OPEN, Capacitor_SMD:C_0201_0603Metric, F.Cu at (34.5, 41.7)
- added C24: C-OPEN, Capacitor_SMD:C_0201_0603Metric, F.Cu at (36.9, 39.6)
- added C24: C-OPEN, Capacitor_SMD:C_0201_0603Metric, F.Cu at (39.3, 43.7)
- added C24: C-OPEN, Capacitor_SMD:C_0201_0603Metric, F.Cu at (35.8, 59.4)
- added C24: C-OPEN, Capacitor_SMD:C_0201_0603Metric, F.Cu at (36.9, 44.7)
- added C24: C-OPEN, Capacitor_SMD:C_0201_0603Metric, F.Cu at (34.5, 42.7)
- added C24: C-OPEN, Capacitor_SMD:C_0201_0603Metric, F.Cu at (35.8, 50.7)
- added C24: C-OPEN, Capacitor_SMD:C_0402_1005Metric, F.Cu at (37.6, 72.9)
- added C24: C-OPEN, Capacitor_SMD:C_0201_0603Metric, F.Cu at (34.5, 44.7)
- added C24: C-OPEN, Capacitor_SMD:C_0201_0603Metric, F.Cu at (43.2, 54.2)
- added C24: C-OPEN, Capacitor_SMD:C_0201_0603Metric, F.Cu at (43.2, 52.4)
- added C24: C-OPEN, Capacitor_SMD:C_0201_0603Metric, F.Cu at (36.9, 45.7)
- added C24: C-OPEN, Capacitor_SMD:C_0201_0603Metric, F.Cu at (40.7, 48.9)
- added C24: C-OPEN, Capacitor_SMD:C_0402_1005Metric, F.Cu at (41.5, 68.2)
- added C24: C-OPEN, Capacitor_SMD:C_0201_0603Metric, F.Cu at (36.9, 40.6)
- added C24: C-OPEN, Capacitor_SMD:C_0402_1005Metric, F.Cu at (34.8, 65.3)
- added C24: C-OPEN, Capacitor_SMD:C_0201_0603Metric, F.Cu at (39.4, 38.7)
- added C24: C-OPEN, Capacitor_SMD:C_0201_0603Metric, F.Cu at (35.8, 48.9)
- added C24: C-OPEN, Capacitor_SMD:C_0201_0603Metric, F.Cu at (40.7, 59.4)
- added C24: C-OPEN, Capacitor_SMD:C_0201_0603Metric, F.Cu at (39.4, 41.7)
- added C24: C-OPEN, Capacitor_SMD:C_0201_0603Metric, F.Cu at (34.5, 45.7)
- added C24: C-OPEN, Capacitor_SMD:C_0201_0603Metric, F.Cu at (43.2, 50.7)
- added C24: C-OPEN, Capacitor_SMD:C_0201_0603Metric, F.Cu at (39.3, 44.7)
- added C24: C-OPEN, Capacitor_SMD:C_0201_0603Metric, F.Cu at (43.2, 48.9)
- added C24: C-OPEN, Capacitor_SMD:C_0201_0603Metric, F.Cu at (38.3, 55.9)
- added C24: C-OPEN, Capacitor_SMD:C_0201_0603Metric, F.Cu at (39.4, 39.6)
- added C24: C-OPEN, Capacitor_SMD:C_0402_1005Metric, F.Cu at (41.5, 70.2)
- added C24: C-OPEN, Capacitor_SMD:C_0201_0603Metric, F.Cu at (39.4, 40.6)
- added C38: 10uF, Capacitor_Tantalum_SMD:CP_EIA-3216-18_Kemet-A, F.Cu at (60.5, 52.3)
- added C48: 100nF, Capacitor_SMD:C_0201_0603Metric, F.Cu at (40.7, 52.4)
- added IC1: XC3S400-4TQ144C, SUNfWGlsaW54X1hDM1MyMDAtNFRRRzE0NEMuemlw:QFP50P2200X2200X160-144N, F.Cu at (57.3, 67.2)
- added J2: Conn_02x10_Top_Bottom, Connector_PinHeader_1.27mm:PinHeader_2x08_P1.27mm_Vertical_SMD, F.Cu at (40.6, 29.7)
- added R8: R-OPEN, Resistor_SMD:R_0402_1005Metric, F.Cu at (77.5, 72.7)
- added U4: STM32F415RGTx, Package_QFP:LQFP-64_10x10mm_P0.5mm, F.Cu at (49.5, 41.1)
- C49: value C-OPEN -> 10uF; footprint Capacitor_SMD:C_0402_1005Metric -> Capacitor_Tantalum_SMD:CP_EIA-3216-18_Kemet-A
- C50: value C-OPEN -> 22pF; footprint Capacitor_SMD:C_0402_1005Metric -> Capacitor_SMD:C_0201_0603Metric; moved to F.Cu
- C51: value C-OPEN -> 10uF; footprint Capacitor_SMD:C_0402_1005Metric -> Capacitor_Tantalum_SMD:CP_EIA-3216-18_Kemet-A; moved to F.Cu
- C53: value 10uF -> 4.7uF; footprint Capacitor_Tantalum_SMD:CP_EIA-3216-18_Kemet-A -> Capacitor_SMD:C_0402_1005Metric
- C54: value 22pF -> 10uF; footprint Capacitor_SMD:C_0201_0603Metric -> Capacitor_Tantalum_SMD:CP_EIA-3216-18_Kemet-A
- C56: value 100nF -> 4.7uF; footprint Capacitor_SMD:C_0201_0603Metric -> Capacitor_SMD:C_0402_1005Metric
- C57, C60: value 4.7uF -> C-OPEN
- C58, C59: value 10uF -> C-OPEN; footprint Capacitor_Tantalum_SMD:CP_EIA-3216-18_Kemet-A -> Capacitor_SMD:C_0402_1005Metric
- C61, R22: moved to F.Cu
- R10: value 100K -> 0; footprint Resistor_SMD:R_0402_1005Metric -> Resistor_SMD:R_0201_0603Metric
- R11: value 100K -> 4.7K
- R12: value R-OPEN -> 330
- R13: value 0 -> 56; footprint Resistor_SMD:R_0201_0603Metric -> Resistor_SMD:R_0402_1005Metric
- R4: value 330 -> 100K
- R5: value 4.7K -> 49.9K
- R7: value 49.9K -> 100K
- U5: value STM32F415RGTx -> AM29LV320DT90EC; footprint Package_QFP:LQFP-64_10x10mm_P0.5mm -> Package_SO:TSOP-I-48_18.4x12mm_P0.5mm
- U6: value AM29LV320DT90EC -> TC74LCX373FT; footprint Package_SO:TSOP-I-48_18.4x12mm_P0.5mm -> Package_SO:SSOP-20_4.4x6.5mm_P0.65mm
- moved R14 71.2 mm to (80.4, 70.7), turned to 0 degrees
- moved R22 60.4 mm to (77.5, 74.7), turned to 0 degrees
- moved U2 59.6 mm to (76.4, 42.6), turned to 0 degrees
- moved Y2 54.7 mm to (69.8, 47.0), turned to 0 degrees
- moved C58 54.3 mm to (37.6, 65.3), turned to 180 degrees
- moved R3 53.3 mm to (74.6, 74.7), turned to 0 degrees
- moved C53 51.9 mm to (34.8, 69.8), turned to 0 degrees
- moved R6 51.1 mm to (74.6, 80.7), turned to 0 degrees
- moved C54 49.4 mm to (78.7, 64.5), turned to 0 degrees
- moved R2 49.0 mm to (74.6, 72.7), turned to 0 degrees
- moved R7 48.1 mm to (77.5, 70.7), turned to 0 degrees
- moved R1 47.7 mm to (74.6, 70.7), turned to 0 degrees
- moved C49 41.6 mm to (66.3, 52.3), turned to 0 degrees
- moved C51 41.3 mm to (34.6, 77.4), turned to 90 degrees
- moved R13 37.3 mm to (77.5, 80.7), turned to 0 degrees
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- renumbered J2 to J3
Connections:
- C49 pad 1: GND -> +3V3
- C49 pad 2: uC_CNTRL1 -> GND
- C50 pad 1: GND -> +1V2
- C50 pad 2: uC_CNTRL4 -> Net-(U3-VFB)
- C51 pad 1: GND -> +3V3
- C51 pad 2: uC_CNTRL2 -> GND
- C52 pad 2: Net-(U2-CC) -> +1V2
- C53 pad 1: +3V3 -> GND
- C53 pad 2: GND -> +2V5
- C54 pad 2: Net-(U3-VFB) -> GND
- C55 pad 1: +3V3 -> +1V2
- C57 pad 1: GND -> /FPGA_CLK1
- C57 pad 2: +2V5 -> GND
- C58 pad 1: +1V2 -> GND
- C58 pad 2: GND -> uC_CNTRL1
- C59 pad 1: +1V2 -> 40MHz_OSC
- C60 pad 2: +1V2 -> uC_CNTRL2
- C61 pad 1: /FPGA_CLK1 -> GND
- C61 pad 2: GND -> uC_CNTRL4
- R10 pad 1: Net-(U2-SET) -> Net-(IC1-IO_L32P_4/GCLK0)
- R10 pad 2: +2V5 -> /FPGA_CLK1
- R11 pad 1: GND -> +3V3
- R11 pad 2: Net-(U2-SET) -> Net-(IC1-IO_L31N_4/INIT_B)
- R12 pad 1: GND -> +2V5
- R12 pad 2: +2V5 -> FPGA_CNTRL3
- R13 pad 1: Net-(U4-IO_L32N_4/GCLK1) -> uC_CNTRL2
- R13 pad 2: /FPGA_CLK1 -> Net-(IC1-CCLK)
- R4 pad 1: +2V5 -> GND
- R4 pad 2: FPGA_CNTRL3 -> Net-(U3-VFB)
- R5 pad 1: +3V3 -> +1V2
- R5 pad 2: Net-(U4-IO_L31N_4/INIT_B) -> Net-(U3-VFB)
- R6 pad 1: GND -> Net-(U2-SET)
- R6 pad 2: Net-(U3-VFB) -> +2V5
- R7 pad 1: +1V2 -> GND
- R7 pad 2: Net-(U3-VFB) -> Net-(U2-SET)
- RN2 pad 1: unconnected-(RN2-R1.1-Pad1) -> INOUT_MCLKO
- RN2 pad 16: unconnected-(RN2-R1.2-Pad16) -> MCLKO
- RN4 pad 2: INOUT_D2 -> INOUT_D4
- RN7 pad 13: MCLKO -> unconnected-(RN7-R4.2-Pad13)
- RN7 pad 4: INOUT_MCLKO -> unconnected-(RN7-R4.1-Pad4)
- TP1 pad 1: FPGA_CNTRL3 -> Net-(IC1-IO_L31N_4/INIT_B)
- TP2 pad 1: Net-(U4-IO_L31N_4/INIT_B) -> FPGA_CNTRL3
- U5 pad 1: +3V3 -> uC_A16
- U5 pad 10: uC_PROG1 -> uC_PROG2
- U5 pad 11: uC_PROG4 -> uC_CNTRL1
- U5 pad 12: GND -> +3V3
- U5 pad 13: +3V3 -> unconnected-(U5-NC-Pad13)
- U5 pad 14: FPGA_CNTRL1 -> +3V3
- U5 pad 16: SERIAL_TX -> uC_A19
- U5 pad 17: SERIAL_RX -> uC_A18
- U5 pad 18: GND -> uC_A8
- U5 pad 19: +3V3 -> uC_A7
- U5 pad 2: uC_A14 -> uC_A15
- U5 pad 20: FPGA_CNTRL2 -> uC_A6
- U5 pad 21: FPGA_CNTRL3 -> uC_A5
- U5 pad 22: uC_CNTRL1 -> uC_A4
- U5 pad 23: uC_CNTRL2 -> uC_A3
- U5 pad 24: uC_AD3 -> uC_A2
- U5 pad 25: uC_AD4 -> uC_A1
- U5 pad 26: unconnected-(U5-PB0-Pad26) -> uC_CNTRL3
- U5 pad 27: unconnected-(U5-PB1-Pad27) -> GND
- U5 pad 28: uC_A9 -> uC_CNTRL2
- U5 pad 29: uC_PROG2 -> uC_AD0
- U5 pad 3: uC_A13 -> uC_A14
- U5 pad 31: Net-(U5-VCAP_1) -> uC_AD1
- U5 pad 32: +3V3 -> unconnected-(U5-DQ9-Pad32)
- U5 pad 33: unconnected-(U5-PB12-Pad33) -> uC_AD2
- U5 pad 35: unconnected-(U5-PB14-Pad35) -> uC_AD3
- U5 pad 37: uC_AD5 -> +3V3
- U5 pad 38: uC_AD6 -> uC_AD4
- U5 pad 39: uC_AD7 -> unconnected-(U5-DQ12-Pad39)
- U5 pad 4: uC_A12 -> uC_A13
- U5 pad 40: uC_A8 -> uC_AD5
- U5 pad 41: uC_A15 -> unconnected-(U5-DQ13-Pad41)
- U5 pad 42: uC_A19 -> uC_AD6
- U5 pad 43: INOUT_PC_CARD_55 -> unconnected-(U5-DQ14-Pad43)
- U5 pad 44: unconnected-(U5-PA11-Pad44) -> uC_AD7
- U5 pad 45: unconnected-(U5-PA12-Pad45) -> uC_A0
- U5 pad 46: unconnected-(U5-PA13-Pad46) -> GND
- U5 pad 47: Net-(U5-VCAP_2) -> GND
- U5 pad 48: +3V3 -> uC_A17
- U5 pad 5: OSC_IN -> uC_A12
- U5 pad 6: OSC_OUT -> uC_A11
- U5 pad 7: NRST -> uC_A10
- U5 pad 8: uC_AD0 -> uC_A9
- U5 pad 9: uC_AD1 -> uC_PROG1
- U6 pad 1: uC_A16 -> GND
- U6 pad 10: uC_PROG2 -> GND
- U6 pad 11: uC_CNTRL1 -> uC_CNTRL4
- U6 pad 12: +3V3 -> uC_A4
- U6 pad 13: unconnected-(U6-NC-Pad13) -> uC_AD4
- U6 pad 14: +3V3 -> uC_AD5
- U6 pad 15: unconnected-(U6-RY/BY#-Pad15) -> uC_A5
- U6 pad 16: uC_A19 -> uC_A6
- U6 pad 17: uC_A18 -> uC_AD6
- U6 pad 18: uC_A8 -> uC_AD7
- U6 pad 2: uC_A15 -> uC_A3
- U6 pad 20: uC_A6 -> +3V3
- U6 pad 3: uC_A14 -> uC_AD3
- U6 pad 4: uC_A13 -> uC_AD2
- U6 pad 5: uC_A12 -> uC_A2
- U6 pad 6: uC_A11 -> uC_A1
- U6 pad 7: uC_A10 -> uC_AD1
- U6 pad 8: uC_A9 -> uC_AD0
- U6 pad 9: uC_PROG1 -> uC_A0
Routing:
- net +2V5: track 120.1 -> 12.5 mm, vias 3 -> 0
- net +1V2: track 122.0 -> 21.7 mm, vias 3 -> 0
- net uC_AD4: track 80.5 -> 0.00 mm, vias 3 -> 0
- net Net-(U2-SET): track 71.0 -> 0.00 mm, vias 2 -> 0
- net uC_A14: track 66.8 -> 0.00 mm, vias 2 -> 0
- net uC_PROG1: track 58.4 -> 0.00 mm, vias 4 -> 0
- net NRST: track 30.6 -> 87.5 mm, vias 0 -> 4
- net uC_AD3: track 51.7 -> 0.00 mm, vias 3 -> 0
- net uC_CNTRL1: track 51.5 -> 0.00 mm, vias 2 -> 0
- net uC_CNTRL2: track 69.4 -> 20.4 mm, vias 3 -> 2
- net FPGA_CNTRL3: track 70.4 -> 21.5 mm, vias 5 -> 2
- net FPGA_TEST_EDGE3: track 0.00 -> 48.4 mm, vias 0 -> 2
- net uC_AD2: track 64.8 -> 16.5 mm, vias 3 -> 2
- net Net-(C73-Pad1): track 47.9 -> 0.00 mm, vias 2 -> 0
- net uC_A13: track 47.3 -> 0.00 mm, vias 2 -> 0
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
Commit message: 12312
Parts:
- moved U4 1.99 mm to (51.4, 41.9)
Routing:
- net Net-(C39-Pad1): track 91.6 -> 0.00 mm, vias 3 -> 0
- net VCC: track 90.1 -> 1.27 mm, vias 5 -> 0
- net NRST: track 87.5 -> 0.00 mm, vias 4 -> 0
- net FPGA_TEST_EDGE3: track 48.4 -> 0.00 mm, vias 2 -> 0
- net FPGA_TEST_EDGE5: track 46.7 -> 0.00 mm, vias 2 -> 0
- net FPGA_TEST_EDGE4: track 45.5 -> 0.00 mm, vias 2 -> 0
- net FPGA_TEST_EDGE2: track 43.4 -> 0.00 mm, vias 3 -> 0
- net Net-(U2-CC): track 43.3 -> 0.00 mm, vias 2 -> 0
- net Net-(U4-VCAP_2): track 43.1 -> 0.00 mm, vias 3 -> 0
- net uC_AD6: track 39.2 -> 0.00 mm, vias 5 -> 0
- net uC_AD7: track 39.2 -> 0.00 mm, vias 3 -> 0
- net FPGA_CNTRL2: track 39.1 -> 0.00 mm, vias 2 -> 0
- net uC_A17: track 36.6 -> 0.00 mm, vias 2 -> 0
- net Net-(U4-VCAP_1): track 34.2 -> 0.00 mm, vias 2 -> 0
- net uC_CNTRL3: track 30.5 -> 0.00 mm, vias 2 -> 0
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Other:
- copper layers 4 -> 6

Commit message: 23623637
Parts:
- removed the C24 at (41.5, 66.2)
- removed the C24 at (40.7, 61.2)
- removed the C24 at (37.6, 71.4)
- removed the C24 at (43.2, 55.9)
- removed the C24 at (40.7, 57.7)
- removed the C24 at (37.6, 72.9)
- removed the C24 at (43.2, 54.2)
- removed the C24 at (43.2, 52.4)
- removed the C24 at (41.5, 68.2)
- removed the C24 at (40.7, 59.4)
- removed the C24 at (43.2, 50.7)
- removed the C24 at (43.2, 48.9)
- removed the C24 at (41.5, 70.2)
- removed C55: 10uF, Capacitor_Tantalum_SMD:CP_EIA-3216-18_Kemet-A
- removed C56: 4.7uF, Capacitor_SMD:C_0402_1005Metric
- removed C57, C58, C59, C60, C61: C-OPEN, Capacitor_SMD:C_0402_1005Metric
- added R18: 0, Resistor_SMD:R_0402_1005Metric, F.Cu at (51.0, 26.9)
- added R19: 0, Resistor_SMD:R_0201_0603Metric, F.Cu at (42.4, 31.8)
- added R20: 47, Resistor_SMD:R_0402_1005Metric, F.Cu at (51.8, 31.5)
- C1, C18, C25, C27, C30: renamed from C24; value C-OPEN -> 10uF; footprint Capacitor_SMD:C_0201_0603Metric -> Capacitor_Tantalum_SMD:CP_EIA-3216-18_Kemet-A
- C24: renamed from C50; value 22pF -> C-OPEN; footprint Capacitor_SMD:C_0201_0603Metric -> Capacitor_SMD:C_0402_1005Metric
- C24: renamed from C48; value 100nF -> C-OPEN
- C24 (x3): footprint Capacitor_SMD:C_0201_0603Metric -> Capacitor_SMD:C_0402_1005Metric
- C24: renamed from C49; value 10uF -> C-OPEN; footprint Capacitor_Tantalum_SMD:CP_EIA-3216-18_Kemet-A -> Capacitor_SMD:C_0402_1005Metric
- C24: footprint Capacitor_SMD:C_0402_1005Metric -> Capacitor_SMD:C_0201_0603Metric
- C24: renamed from C33; value 10uF -> C-OPEN; footprint Capacitor_Tantalum_SMD:CP_EIA-3216-18_Kemet-A -> Capacitor_SMD:C_0201_0603Metric
- C24: renamed from C51; value 10uF -> C-OPEN; footprint Capacitor_Tantalum_SMD:CP_EIA-3216-18_Kemet-A -> Capacitor_SMD:C_0201_0603Metric
- C24: renamed from C52; value 100nF -> C-OPEN; footprint Capacitor_SMD:C_0201_0603Metric -> Capacitor_SMD:C_0402_1005Metric
- C24: value C-OPEN -> 100nF
- C24: renamed from C53; value 4.7uF -> C-OPEN
- C24: renamed from C54; value 10uF -> C-OPEN; footprint Capacitor_Tantalum_SMD:CP_EIA-3216-18_Kemet-A -> Capacitor_SMD:C_0201_0603Metric
- C26: renamed from C24; value C-OPEN -> 22pF
- C28, C4: renamed from C24; value C-OPEN -> 100nF
- C29, C5: renamed from C24; value C-OPEN -> 4.7uF; footprint Capacitor_SMD:C_0201_0603Metric -> Capacitor_SMD:C_0402_1005Metric
- C3: renamed from C24; value C-OPEN -> 1nF
- C35: value 1nF -> 10uF; footprint Capacitor_SMD:C_0201_0603Metric -> Capacitor_Tantalum_SMD:CP_EIA-3216-18_Kemet-A
- C36: value 100nF -> 4.7uF; footprint Capacitor_SMD:C_0201_0603Metric -> Capacitor_SMD:C_0402_1005Metric
- C37: value 4.7uF -> C-OPEN
- C38: value 10uF -> C-OPEN; footprint Capacitor_Tantalum_SMD:CP_EIA-3216-18_Kemet-A -> Capacitor_SMD:C_0402_1005Metric
- C40, C41: renamed from C24; footprint Capacitor_SMD:C_0201_0603Metric -> Capacitor_SMD:C_0402_1005Metric
- J1: value MEC1-108-01-S-D-RA1-SL -> Conn_02x04_Top_Bottom; footprint Connector_PinSocket_1.27mm:PinSocket_2x08_P1.27mm_Vertical_SMD -> Connector_PinHeader_1.27mm:PinHeader_2x04_P1.27mm_Vertical
- J2: value Conn_02x10_Top_Bottom -> MEC1-108-01-S-D-RA1-SL; footprint Connector_PinHeader_1.27mm:PinHeader_2x08_P1.27mm_Vertical_SMD -> Connector_PinSocket_1.27mm:PinSocket_2x08_P1.27mm_Vertical_SMD; moved to B.Cu
- R14: value 10K -> 330
- R15: value 0 -> 56
- R17: value 47 -> 10K
- R22: renamed from R12; value 330 -> 56
- R22: renamed from R16; value 0 -> 56; footprint Resistor_SMD:R_0201_0603Metric -> Resistor_SMD:R_0402_1005Metric
- moved R14 55.3 mm to (39.0, 34.0)
- moved R22 54.2 mm to (53.8, 25.9)
- moved R11 52.6 mm to (43.0, 37.0)
- moved C24 51.1 mm to (56.0, 91.0)
- moved C24 50.5 mm to (48.0, 95.0)
- moved C28 49.6 mm to (64.0, 95.0)
- moved C39 49.3 mm to (79.0, 90.0)
- moved C24 47.2 mm to (35.3, 30.2)
- moved C5 47.0 mm to (78.5, 26.2)
- moved R17 46.5 mm to (34.0, 71.0)
- moved C24 45.6 mm to (36.0, 96.0)
- moved C36 45.4 mm to (40.0, 96.0)
- moved Y2 44.7 mm to (35.8, 76.0)
- moved C24 44.5 mm to (51.0, 85.0)
- moved C24 43.5 mm to (80.0, 46.0)
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- renumbered C24 to C39, R13 to R22
Connections:
- C1 pad 1: +3V3 -> VCC
- C18 pad 1: +3V3 -> VCC
- C24 pad 1: +2V5 -> +1V2 (x2)
- C24 pad 1: +1V2 -> +3V3 (x6)
- C24 pad 1: +1V2 -> Net-(U4-VCAP_2)
- C24 pad 2: Net-(U3-VFB) -> GND
- C24 pad 1: GND -> NRST
- C24 pad 2: Net-(U2-CC) -> GND
- C24 pad 1: +1V2 -> uC_CNTRL2
- C24 pad 1: +3V3 -> +2V5 (x4)
- C24 pad 1: +3V3 -> Net-(U4-VCAP_1)
- C24 pad 1: +3V3 -> Net-(C19-Pad1)
- C24 pad 1: +3V3 -> +1V2
- C24 pad 1: VCC -> +1V2
- C24 pad 1: GND -> OSC_IN
- C24 pad 2: +1V2 -> GND
- C24 pad 1: +3V3 -> GND
- C24 pad 2: GND -> Net-(U2-CC)
- C24 pad 1: GND -> Net-(C53-Pad1)
- C24 pad 2: +2V5 -> GND
- C25 pad 1: +2V5 -> +3V3
- C26 pad 1: +2V5 -> +1V2
- C26 pad 2: GND -> Net-(U3-VFB)
- C27 pad 1: +2V5 -> +3V3
- C28 pad 1: +2V5 -> GND
- C28 pad 2: GND -> +1V2
- C29 pad 1: +2V5 -> GND
- C29 pad 2: GND -> +2V5
- C3 pad 1: +3V3 -> GND
- C3 pad 2: GND -> Net-(C3-Pad2)
- C30 pad 1: +2V5 -> +1V2
- C35 pad 1: GND -> +1V2
- C35 pad 2: Net-(C35-Pad2) -> GND
- C36 pad 2: VCC -> +1V2
- C37 pad 1: GND -> /FPGA_CLK1
- C37 pad 2: VCC -> GND
- C38 pad 1: VCC -> GND
- C38 pad 2: GND -> uC_CNTRL1
- C39 pad 1: Net-(C39-Pad1) -> 40MHz_OSC
- C4 pad 1: +3V3 -> GND
- C4 pad 2: GND -> VCC
- C40 pad 1: +1V2 -> GND
- C40 pad 2: GND -> uC_CNTRL2
- C41 pad 1: +1V2 -> GND
- C41 pad 2: GND -> uC_CNTRL4
- C5 pad 1: +3V3 -> GND
- C5 pad 2: GND -> VCC
- J1 pad 2: GND -> Net-(J1-Pin_2)
- J1 pad 3: SERIAL_RX -> Net-(J1-Pin_3)
- J1 pad 4: SERIAL_TX -> Net-(IC1-TDO)
- J1 pad 5: unconnected-(J1-Pad5) -> GND
- J1 pad 6: unconnected-(J1-Pad6) -> Net-(J1-Pin_6)
- J1 pad 7: FPGA_TEST_EDGE1 -> unconnected-(J1-Pin_7-Pad7)
- J1 pad 8: FPGA_TEST_EDGE2 -> unconnected-(J1-Pin_8-Pad8)
- J2 pad 1: unconnected-(J2-Pin_1-Pad1) -> +3V3
- J2 pad 10: unconnected-(J2-Pin_10-Pad10) -> FPGA_TEST_EDGE4
- J2 pad 11: unconnected-(J2-Pin_11-Pad11) -> FPGA_TEST_EDGE5
- J2 pad 12: unconnected-(J2-Pin_12-Pad12) -> FPGA_TEST_EDGE6
- J2 pad 13: unconnected-(J2-Pin_13-Pad13) -> uC_PROG1
- J2 pad 14: unconnected-(J2-Pin_14-Pad14) -> NRST
- J2 pad 15: unconnected-(J2-Pin_15-Pad15) -> uC_PROG2
- J2 pad 16: unconnected-(J2-Pin_16-Pad16) -> uC_PROG4
- J2 pad 2: unconnected-(J2-Pin_2-Pad2) -> GND
- J2 pad 3: unconnected-(J2-Pin_3-Pad3) -> SERIAL_RX
- J2 pad 4: unconnected-(J2-Pin_4-Pad4) -> SERIAL_TX
- J2 pad 7: unconnected-(J2-Pin_7-Pad7) -> FPGA_TEST_EDGE1
- J2 pad 8: unconnected-(J2-Pin_8-Pad8) -> FPGA_TEST_EDGE2
- J2 pad 9: unconnected-(J2-Pin_9-Pad9) -> FPGA_TEST_EDGE3
- R1 pad 2: Net-(C35-Pad2) -> Net-(C3-Pad2)
- R14 pad 1: NRST -> +2V5
- R14 pad 2: +3V3 -> FPGA_CNTRL3
- R15 pad 1: Net-(J3-CD1#) -> uC_CNTRL2
- R15 pad 2: GND -> Net-(IC1-CCLK)
- R17 pad 1: OSC_OUT -> NRST
- R17 pad 2: Net-(C73-Pad1) -> +3V3
- R2 pad 2: Net-(C39-Pad1) -> Net-(C19-Pad1)
- R22 pad 1: uC_CNTRL2 -> Net-(J1-Pin_3)
- R22 pad 2: Net-(IC1-CCLK) -> Net-(IC1-TCK)
- R22 pad 1: +2V5 -> Net-(J1-Pin_2)
- R22 pad 2: FPGA_CNTRL3 -> Net-(IC1-TMS)
- R22 pad 1: GND -> TDI
- R22 pad 2: Net-(J3-CD2#) -> Net-(J1-Pin_6)
- Y1 pad 3: Net-(C39-Pad1) -> Net-(C19-Pad1)
- Y2 pad 3: Net-(C73-Pad1) -> Net-(C53-Pad1)
Routing:
- net GND: track 89.5 -> 0.00 mm, vias 38 -> 0
- net FPGA_TEST_EDGE6: track 42.5 -> 0.00 mm, vias 2 -> 0
- net Net-(J3-CD2#): track 41.6 -> 0.00 mm, vias 2 -> 0
- net Net-(J3-CD1#): track 26.8 -> 0.00 mm, vias 2 -> 0
- net +1V2: track 21.7 -> 0.00 mm
- net uC_A10: track 16.4 -> 0.00 mm, vias 2 -> 0
- net uC_A16: track 15.3 -> 0.00 mm, vias 2 -> 0
- net INOUT_A5: track 14.0 -> 0.00 mm
- net +2V5: track 12.5 -> 0.00 mm
- net MDI3: track 10.8 -> 0.00 mm
- net IREQ#: track 10.8 -> 0.00 mm
- net +3V3: track 1.78 -> 0.00 mm, vias 1 -> 0
- net VCC: track 1.27 -> 0.00 mm
Other:
- copper layers 6 -> 4

Commit message: 2234545
Parts:
- removed RN7: 8 x 180R, Resistor_SMD:R_Cat16-8
- C2: renamed from C24; value C-OPEN -> 1nF; footprint Capacitor_SMD:C_0402_1005Metric -> Capacitor_SMD:C_0201_0603Metric
- C24: renamed from C3; value 1nF -> C-OPEN; footprint Capacitor_SMD:C_0201_0603Metric -> Capacitor_SMD:C_0402_1005Metric
- IC1: footprint SUNfWGlsaW54X1hDM1MyMDAtNFRRRzE0NEMuemlw:QFP50P2200X2200X160-144N -> QFP50P2200X2200X160-144N:QFP50P2200X2200X160-144N
- J2: value MEC1-108-01-S-D-RA1-SL -> Conn_02x04_Top_Bottom; footprint Connector_PinSocket_1.27mm:PinSocket_2x08_P1.27mm_Vertical_SMD -> Connector_PinHeader_1.27mm:PinHeader_2x04_P1.27mm_Vertical; moved to F.Cu
- R2: value 47 -> 220K
- R3: value 220K -> 47
- moved RN5 34.6 mm to (77.0, 91.7)
- moved RN3 29.5 mm to (38.1, 91.7)
- moved C37 27.0 mm to (80.3, 85.4)
- moved J2 24.6 mm to (53.8, 51.3)
- moved Y2 23.9 mm to (51.0, 57.7)
- moved C24 22.3 mm to (76.4, 82.1)
- moved C36 21.6 mm to (35.0, 74.9)
- moved R15 21.0 mm to (78.0, 77.5)
- moved RN2 20.5 mm to (69.1, 91.7)
- moved C28 20.0 mm to (79.9, 82.8)
- moved C24 19.9 mm to (75.1, 78.0)
- moved RN4 17.6 mm to (61.2, 91.7)
- moved C24 17.3 mm to (35.0, 78.8)
- moved RN1 16.3 mm to (53.3, 91.7)
- moved C24 16.1 mm to (35.0, 82.8)
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Connections:
- C2 pad 1: +3V3 -> GND
- C2 pad 2: GND -> Net-(C2-Pad2)
- C24 pad 1: GND -> +3V3
- C24 pad 2: Net-(C3-Pad2) -> GND
- IC1 pad 10: INOUT_A5 -> INOUT_A4
- IC1 pad 105: INOUT_RESET -> INOUT_MCLKI
- IC1 pad 107: INOUT_WE# -> unconnected-(IC1-IO_L01P_2/VRN_2-Pad107)
- IC1 pad 108: INOUT_MCLKI -> unconnected-(IC1-IO_L01N_2/VRP_2-Pad108)
- IC1 pad 109: unconnected-(IC1-TDO-Pad109) -> Net-(IC1-TDO)
- IC1 pad 11: INOUT_A4 -> INOUT_A3
- IC1 pad 110: unconnected-(IC1-TCK-Pad110) -> Net-(IC1-TCK)
- IC1 pad 111: unconnected-(IC1-TMS-Pad111) -> Net-(IC1-TMS)
- IC1 pad 12: INOUT_A3 -> INOUT_A2
- IC1 pad 129: FPGA_TEST_EDGE6 -> unconnected-(IC1-IO_L31P_0/VREF_0-Pad129)
- IC1 pad 13: INOUT_A2 -> INOUT_A1
- IC1 pad 130: FPGA_TEST_EDGE5 -> INOUT_MISTRT
- IC1 pad 131: FPGA_TEST_EDGE4 -> INOUT_IOWR#
- IC1 pad 132: FPGA_TEST_EDGE3 -> INOUT_IORD#
- IC1 pad 135: FPGA_TEST_EDGE2 -> INOUT_RESET
- IC1 pad 137: FPGA_TEST_EDGE1 -> INOUT_WE#
- IC1 pad 14: INOUT_A1 -> INOUT_A0
- IC1 pad 144: unconnected-(IC1-TDI-Pad144) -> TDI
- IC1 pad 15: INOUT_A0 -> INOUT_INPACK#
- IC1 pad 17: unconnected-(IC1-IO_L40P_7-Pad17) -> INOUT_REG#
- IC1 pad 20: INOUT_INPACK# -> unconnected-(IC1-IO_L40P_6/VREF_6-Pad20)
- IC1 pad 21: INOUT_REG# -> INOUT_MOVAL
- IC1 pad 23: INOUT_MOVAL -> INOUT_MIVAL
- IC1 pad 24: INOUT_MIVAL -> INOUT_MDO7
- IC1 pad 25: INOUT_MDO7 -> INOUT_MDO6
- IC1 pad 26: INOUT_MDO6 -> INOUT_MDO5
- IC1 pad 27: INOUT_MDO5 -> INOUT_MDO4
- IC1 pad 28: INOUT_MDO4 -> INOUT_MDO3
- IC1 pad 30: INOUT_MDO3 -> INOUT_MDO2
- IC1 pad 31: INOUT_MDO2 -> INOUT_MDO1
- IC1 pad 32: INOUT_MDO1 -> INOUT_MDO0
- IC1 pad 33: INOUT_MDO0 -> INOUT_IREQ#
- IC1 pad 5: unconnected-(IC1-IO_L20P_7-Pad5) -> INOUT_MCLKO
- IC1 pad 53: INOUT_MCLKI -> unconnected-(IC1-IO_L32N_5/GCLK3-Pad53)
- IC1 pad 6: INOUT_MCLKO -> INOUT_A7
- IC1 pad 7: INOUT_A7 -> INOUT_A6
- IC1 pad 77: INOUT_IREQ# -> INOUT_D0
- IC1 pad 78: INOUT_D0 -> INOUT_D1
- IC1 pad 79: INOUT_D1 -> INOUT_D2
- IC1 pad 8: INOUT_A6 -> INOUT_A5
- IC1 pad 80: INOUT_D2 -> INOUT_D3
- IC1 pad 82: INOUT_D3 -> INOUT_D4
- IC1 pad 83: INOUT_D4 -> INOUT_D5
- IC1 pad 84: INOUT_D5 -> unconnected-(IC1-IO_L23P_3/VREF_3-Pad84)
- IC1 pad 90: INOUT_CE1# -> unconnected-(IC1-IO_L40N_3/VREF_3-Pad90)
- IC1 pad 92: INOUT_MISTRT -> unconnected-(IC1-IO_L40P_2/VREF_2-Pad92)
- IC1 pad 93: INOUT_IOWR# -> INOUT_CE1#
- IC1 pad 95: INOUT_IORD# -> INOUT_MDI0
- IC1 pad 96: INOUT_MDI0 -> INOUT_MDI1
- IC1 pad 97: INOUT_MDI1 -> INOUT_MDI2
- IC1 pad 98: INOUT_MDI2 -> unconnected-(IC1-IO_L23N_2/VREF_2-Pad98)
- J1 pad 1: +3V3 -> Net-(J1-Pin_1)
- J1 pad 6: Net-(J1-Pin_6) -> GND
- J1 pad 7: unconnected-(J1-Pin_7-Pad7) -> GND
- J1 pad 8: unconnected-(J1-Pin_8-Pad8) -> +3V3
- J2 pad 2: GND -> SERIAL_RX
- J2 pad 3: SERIAL_RX -> uC_PROG1
- J2 pad 4: SERIAL_TX -> uC_PROG2
- J2 pad 5: unconnected-(J2-Pad5) -> GND
- J2 pad 6: unconnected-(J2-Pad6) -> SERIAL_TX
- J2 pad 7: FPGA_TEST_EDGE1 -> NRST
- J2 pad 8: FPGA_TEST_EDGE2 -> uC_PROG4
- R1 pad 2: Net-(C3-Pad2) -> Net-(C2-Pad2)
- R2 pad 1: 40MHz_OSC -> GND
- R2 pad 2: Net-(C19-Pad1) -> Net-(U3-SHDN/RT)
- R22 pad 2: Net-(J1-Pin_6) -> Net-(J1-Pin_1)
- R3 pad 1: GND -> 40MHz_OSC
- R3 pad 2: Net-(U3-SHDN/RT) -> Net-(C19-Pad1)
- RN1 pad 1: INOUT_MOSTRT -> INOUT_MCLKI
- RN1 pad 10: MDO2 -> MCLKO
- RN1 pad 11: D2 -> A6
- RN1 pad 12: MDO1 -> MDI7
- RN1 pad 13: D1 -> A7
- RN1 pad 14: MDO0 -> MDI6
- RN1 pad 15: D0 -> MDI5
- RN1 pad 16: MOSTRT -> MCLKI
- RN1 pad 2: INOUT_D0 -> INOUT_MDI5
- RN1 pad 3: INOUT_MDO0 -> INOUT_MDI6
- RN1 pad 4: INOUT_D1 -> INOUT_A7
- RN1 pad 5: INOUT_MDO1 -> INOUT_MDI7
- RN1 pad 6: INOUT_D2 -> INOUT_A6
- RN1 pad 7: INOUT_MDO2 -> INOUT_MCLKO
- RN1 pad 8: unconnected-(RN1-R8.1-Pad8) -> INOUT_A5
- RN1 pad 9: unconnected-(RN1-R8.2-Pad9) -> A5
- RN2 pad 1: INOUT_MCLKO -> unconnected-(RN2-R1.1-Pad1)
- RN2 pad 10: RESET -> IOWR#
- RN2 pad 11: A5 -> IORD#
- RN2 pad 12: A6 -> OE#
- RN2 pad 13: MDI7 -> MDO7
- RN2 pad 14: A7 -> CE1#
- RN2 pad 15: MDI6 -> MDO6
- RN2 pad 16: MCLKO -> unconnected-(RN2-R1.2-Pad16)
- RN2 pad 2: INOUT_MDI6 -> INOUT_MDO6
- RN2 pad 3: INOUT_A7 -> INOUT_CE1#
- RN2 pad 4: INOUT_MDI7 -> INOUT_MDO7
- RN2 pad 5: INOUT_A6 -> INOUT_OE#
- RN2 pad 6: INOUT_A5 -> INOUT_IORD#
- RN2 pad 7: INOUT_RESET -> INOUT_IOWR#
- RN2 pad 8: INOUT_A4 -> INOUT_MISTRT
- RN2 pad 9: A4 -> MISTRT
- RN3 pad 1: unconnected-(RN3-R1.1-Pad1) -> INOUT_A0
- RN3 pad 10: unconnected-(RN3-R7.2-Pad10) -> D2
- RN3 pad 11: MDI0 -> MDO1
- RN3 pad 12: unconnected-(RN3-R5.2-Pad12) -> D1
- RN3 pad 13: MISTRT -> MDO0
- RN3 pad 14: unconnected-(RN3-R3.2-Pad14) -> D0
- RN3 pad 15: IOWR# -> MOSTRT
- RN3 pad 16: unconnected-(RN3-R1.2-Pad16) -> A0
- RN3 pad 2: INOUT_IOWR# -> INOUT_MOSTRT
- RN3 pad 3: unconnected-(RN3-R3.1-Pad3) -> INOUT_D0
- RN3 pad 4: INOUT_MISTRT -> INOUT_MDO0
- RN3 pad 5: unconnected-(RN3-R5.1-Pad5) -> INOUT_D1
- RN3 pad 6: INOUT_MDI0 -> INOUT_MDO1
- RN3 pad 7: unconnected-(RN3-R7.1-Pad7) -> INOUT_D2
- RN3 pad 8: INOUT_MDI1 -> INOUT_MDO2
- RN3 pad 9: MDI1 -> MDO2
- RN4 pad 1: INOUT_D3 -> INOUT_MDI0
- RN4 pad 10: MDO5 -> MIVAL
- RN4 pad 11: D6 -> MDI3
- RN4 pad 12: MDO4 -> IREQ#
- RN4 pad 13: D5 -> MDI2
- RN4 pad 14: MDO3 -> WE#
- RN4 pad 15: D4 -> MDI1
- RN4 pad 16: D3 -> MDI0
- RN4 pad 2: INOUT_D4 -> INOUT_MDI1
- RN4 pad 3: INOUT_MDO3 -> INOUT_WE#
- RN4 pad 4: INOUT_D5 -> INOUT_MDI2
- RN4 pad 5: INOUT_MDO4 -> INOUT_IREQ#
- RN4 pad 6: INOUT_D6 -> INOUT_MDI3
- RN4 pad 7: INOUT_MDO5 -> INOUT_MIVAL
- RN4 pad 8: INOUT_D7 -> INOUT_MDI4
- RN4 pad 9: D7 -> MDI4
- RN5 pad 1: unconnected-(RN5-R1.1-Pad1) -> INOUT_D3
- RN5 pad 10: MOVAL -> MDO5
- RN5 pad 11: A1 -> D6
- RN5 pad 12: REG# -> MDO4
- RN5 pad 13: A2 -> D5
- RN5 pad 14: INPACK# -> MDO3
- RN5 pad 15: A3 -> D4
- RN5 pad 16: unconnected-(RN5-R1.2-Pad16) -> D3
- RN5 pad 2: INOUT_A3 -> INOUT_D4
- RN5 pad 3: INOUT_INPACK# -> INOUT_MDO3
- RN5 pad 4: INOUT_A2 -> INOUT_D5
- RN5 pad 5: INOUT_REG# -> INOUT_MDO4
- RN5 pad 6: INOUT_A1 -> INOUT_D6
- RN5 pad 7: INOUT_MOVAL -> INOUT_MDO5
- RN5 pad 8: INOUT_A0 -> INOUT_D7
- RN5 pad 9: A0 -> D7
- RN6 pad 1: INOUT_WE# -> INOUT_RESET
- RN6 pad 10: MCLKI -> A1
- RN6 pad 11: MDI4 -> REG#
- RN6 pad 12: MIVAL -> A2
- RN6 pad 13: MDI3 -> INPACK#
- RN6 pad 14: IREQ# -> A3
- RN6 pad 15: MDI2 -> A4
- RN6 pad 16: WE# -> RESET
- RN6 pad 2: INOUT_MDI2 -> INOUT_A4
- RN6 pad 3: INOUT_IREQ# -> INOUT_A3
- RN6 pad 4: INOUT_MDI3 -> INOUT_INPACK#
- RN6 pad 5: INOUT_MIVAL -> INOUT_A2
- RN6 pad 6: INOUT_MDI4 -> INOUT_REG#
- RN6 pad 7: INOUT_MCLKI -> INOUT_A1
- RN6 pad 8: INOUT_MDI5 -> INOUT_MOVAL
- RN6 pad 9: MDI5 -> MOVAL
Routing:
- net GND: track 0.00 -> 48.9 mm, vias 0 -> 37
- net MDI6: track 0.00 -> 11.1 mm, vias 0 -> 2
- net MDO2: track 0.00 -> 7.34 mm
- net D2: track 0.00 -> 7.27 mm
- net MIVAL: track 0.00 -> 7.26 mm
- net MDO1: track 0.00 -> 7.20 mm
- net MDI4: track 0.00 -> 7.19 mm
- net D1: track 0.00 -> 7.13 mm
- net MDO0: track 0.00 -> 7.07 mm
- net D4: track 0.00 -> 7.02 mm
- net D0: track 0.00 -> 7.00 mm
- net MDO3: track 0.00 -> 6.96 mm
- net MOSTRT: track 0.00 -> 6.93 mm
- net D5: track 0.00 -> 6.89 mm
- net A0: track 0.00 -> 6.86 mm
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