File: CAM_XILINX_STM/com_1300/com_1300.kicad_pcb (KiCad board)
At the start: 4 copper layers, 50 x 75.9 mm, 104 parts, among them IC1 XC3S400-4TQ144C, IC2 SN74CBTD3384CDBR, IC3 SN74CBTD3384CDBR, IC4 SN74CBTD3384CDBR, IC5 SN74CBTD3384CDBR, J1 Conn_02x04_Top_Bottom, J2 Conn_02x04_Top_Bottom, J3 Conn_02x03_Top_Bottom, J4 9-68RD-0.635SF, U1 LT1963AxST-3.3, U2 LP3982IMM-ADJ, U3 LTC3411EMS, U4 STM32F415RGTx, U5 AM29LV320DT90EC, U6 TC74LCX373FT, Y1 40mHZ, Y2 16mHz

Commit message: fdsdsf
Parts:
- C2, C24 (x24), C26, C28, C4: footprint Capacitor_SMD:C_0402_1005Metric -> Capacitor_SMD:C_0201_0603Metric
- C24 (x5): footprint Capacitor_SMD:C_0402_1005Metric -> Capacitor_SMD:C_0201_0603Metric; moved to B.Cu
- C38: value C-OPEN -> 100 nF
- IC1: footprint QFP50P2200X2200X160-144N:QFP50P2200X2200X160-144N -> SUNfWGlsaW54X1hDM1MyMDAtNFRRRzE0NEMuemlw:QFP50P2200X2200X160-144N
- moved R8 37.1 mm to (40.8, 65.6)
- moved C29 37.1 mm to (40.9, 67.0)
- moved R6 37.1 mm to (34.7, 67.1)
- moved R7 37.1 mm to (36.1, 67.1)
- moved U2 37.1 mm to (40.2, 70.3)
- moved C24 37.1 mm to (34.3, 69.6)
- moved C5 36.5 mm to (34.8, 74.3)
- moved C24 34.9 mm to (39.0, 63.5)
- moved C24 34.9 mm to (38.0, 62.3)
- moved R3 34.9 mm to (40.0, 62.3)
- moved Y1 29.3 mm to (38.8, 57.0)
- moved C24 11.8 mm to (67.4, 46.4), turned to 180 degrees
- moved C24 11.8 mm to (67.4, 44.5), turned to 180 degrees
- moved C24 11.8 mm to (67.4, 45.5), turned to 180 degrees
- moved C24 11.7 mm to (67.3, 42.6), turned to 180 degrees
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Routing:
- net GND: track 11.3 -> 0.00 mm, vias 2 -> 0
- net Net-(J4-CD1#): track 10.3 -> 0.00 mm, vias 2 -> 0
- net MDO2: track 6.89 -> 0.00 mm
- net D2: track 6.72 -> 0.00 mm
- net MDO1: track 6.65 -> 0.00 mm
- net D1: track 6.55 -> 0.00 mm
- net MIVAL: track 6.50 -> 0.00 mm
- net MDO0: track 6.48 -> 0.00 mm
- net MDI4: track 6.43 -> 0.00 mm
- net D0: track 6.41 -> 0.00 mm
- net MOSTRT: track 6.35 -> 0.00 mm
- net A0: track 6.28 -> 0.00 mm
- net D4: track 6.17 -> 0.00 mm
- net MDO3: track 6.10 -> 0.00 mm
- net D5: track 6.03 -> 0.00 mm
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- added copper zone on F.Cu, net (none)
- added copper zone on F.Cu, net GND
- removed copper zone on In2.Cu, net +3V3
- removed copper zone on In1.Cu, net GND

Commit message: 23423
Parts:
- added R21: 10K, Resistor_SMD:R_0402_1005Metric, F.Cu at (56.6, 43.7)
- IC1: footprint SUNfWGlsaW54X1hDM1MyMDAtNFRRRzE0NEMuemlw:QFP50P2200X2200X160-144N -> QFP50P2200X2200X160-144N:QFP50P2200X2200X160-144N
Connections:
- C1 pad 2: GND -> BOOT0
- C18 pad 2: GND -> BOOT0
- C2 pad 1: GND -> BOOT0
- C24 pad 2: GND -> BOOT0 (x35)
- C24 pad 1: GND -> BOOT0
- C25 pad 2: GND -> BOOT0
- C27 pad 2: GND -> BOOT0
- C28 pad 1: GND -> BOOT0
- C29 pad 1: GND -> BOOT0
- C30 pad 2: GND -> BOOT0
- C35 pad 2: GND -> BOOT0
- C36 pad 1: GND -> BOOT0
- C37 pad 2: GND -> BOOT0
- C38 pad 1: GND -> BOOT0
- C39 pad 2: GND -> BOOT0
- C4 pad 1: GND -> BOOT0
- C40 pad 1: GND -> BOOT0
- C41 pad 1: GND -> BOOT0
- C5 pad 1: GND -> BOOT0
- C55 pad 1: GND -> BOOT0
- C56 pad 1: GND -> BOOT0
- C57 pad 1: GND -> BOOT0
- C58 pad 1: GND -> BOOT0
- IC1 pad 101: GND -> BOOT0
- IC1 pad 114: GND -> BOOT0
- IC1 pad 117: GND -> BOOT0
- IC1 pad 136: GND -> BOOT0
- IC1 pad 139: GND -> BOOT0
- IC1 pad 16: GND -> BOOT0
- IC1 pad 22: GND -> BOOT0
- IC1 pad 29: GND -> BOOT0
- IC1 pad 38: GND -> BOOT0
- IC1 pad 42: GND -> BOOT0
- IC1 pad 45: GND -> BOOT0
- IC1 pad 64: GND -> BOOT0
- IC1 pad 67: GND -> BOOT0
- IC1 pad 81: GND -> BOOT0
- IC1 pad 88: GND -> BOOT0
- IC1 pad 9: GND -> BOOT0
- IC1 pad 94: GND -> BOOT0
- IC2 pad 12: GND -> BOOT0
- IC3 pad 12: GND -> BOOT0
- IC4 pad 12: GND -> BOOT0
- IC5 pad 12: GND -> BOOT0
- J1 pad 5: GND -> BOOT0
- J1 pad 6: GND -> BOOT0
- J1 pad 7: GND -> BOOT0
- J2 pad 5: GND -> BOOT0
- J3 pad 4: GND -> BOOT0
- J4 pad 1: GND -> BOOT0
- J4 pad 34: GND -> BOOT0
- J4 pad 35: GND -> BOOT0
- J4 pad 68: GND -> BOOT0
- R18 pad 2: GND -> BOOT0
- R19 pad 1: GND -> BOOT0
- R2 pad 1: GND -> BOOT0
- R4 pad 1: GND -> BOOT0
- R7 pad 1: GND -> BOOT0
- R8 pad 1: GND -> BOOT0
- U1 pad 2: GND -> BOOT0
- U2 pad 3: GND -> BOOT0
- U3 pad 11: GND -> BOOT0
- U3 pad 2: GND -> BOOT0
- U3 pad 3: GND -> BOOT0
- U3 pad 5: GND -> BOOT0
- U4 pad 12: GND -> BOOT0
- U4 pad 18: GND -> BOOT0
- U4 pad 60: BOOT0 -> Net-(U4-BOOT0)
- U4 pad 63: GND -> BOOT0
- U5 pad 27: GND -> BOOT0
- U5 pad 46: GND -> BOOT0
- U5 pad 47: GND -> BOOT0
- U6 pad 1: GND -> BOOT0
- U6 pad 10: GND -> BOOT0
- Y1 pad 2: GND -> BOOT0
- Y1 pad 4: GND -> BOOT0
- Y2 pad 2: GND -> BOOT0
- Y2 pad 4: GND -> BOOT0
Routing:
- added copper zone on F.Cu, net BOOT0
- removed copper zone on F.Cu, net GND

Commit message: 32244
Parts:
- removed C56, C57, C58: 100 nF, Capacitor_SMD:C_0201_0603Metric
- removed TP1, TP2: TestPoint_Small, TestPoint:TestPoint_Pad_D1.0mm
- added JTAG1: Conn_02x04_Top_Bottom, Connector_PinHeader_1.27mm:PinHeader_2x04_P1.27mm_Vertical, F.Cu at (76.2, 71.7)
- added R22: 47, Resistor_SMD:R_0402_1005Metric, F.Cu at (41.8, 52.7)
- C20: renamed from C24; value C-OPEN -> 100nF
- C21, C6: renamed from C24; value C-OPEN -> 10uF
- C22: renamed from C24; value C-OPEN -> 22pF
- C24: renamed from C26; value 22pF -> C-OPEN
- C24: renamed from C55; value 100 nF -> C-OPEN
- C24: renamed from C25; value 10uF -> C-OPEN
- C24: renamed from C18; value 10uF -> C-OPEN
- C24: value 100nF -> C-OPEN
- C37, C39: value C-OPEN -> 100 nF
- C42, C50, C52: renamed from C24; value C-OPEN -> 100 nF
- J1: value Conn_02x04_Top_Bottom -> Conn_01x02
- J2: value Conn_02x04_Top_Bottom -> Conn_02x03_Top_Bottom
- J3: value Conn_02x03_Top_Bottom -> Conn_02x04_Top_Bottom
- J4: value 9-68RD-0.635SF -> Conn_02x03_Top_Bottom
- R11: value 4.7K -> 0
- R12: renamed from R22; value 56 -> 4.7K
- R15: value 56 -> 4,7K
- R19: value 0 -> 10K
- R20: value 47 -> 0
- R21: value 10K -> 33
- R22: renamed from R14; value 330 -> 56
- R9: renamed from R22; value 56 -> 4,7K
- U4: value STM32F415RGTx -> XCF02SVOG20C
- U5: value AM29LV320DT90EC -> STM32F415RGTx
- U6: value TC74LCX373FT -> W25Q64BVSSIG
Connections:
- C1 pad 2: BOOT0 -> GND
- C2 pad 1: BOOT0 -> GND
- C20 pad 1: +2V5 -> GND
- C20 pad 2: BOOT0 -> Net-(U2-CC)
- C21 pad 1: +2V5 -> +3V3
- C21 pad 2: BOOT0 -> GND
- C22 pad 1: +2V5 -> +1V2
- C22 pad 2: BOOT0 -> Net-(U3-VFB)
- C24 pad 1: +1V2 -> +2V5
- C24 pad 2: Net-(U3-VFB) -> GND
- C24 pad 1: Net-(U4-VCAP_1) -> Net-(U5-VCAP_1)
- C24 pad 2: BOOT0 -> GND (x30)
- C24 pad 1: +3V3 -> Net-(U5-VCAP_2)
- C24 pad 1: BOOT0 -> Net-(C55-Pad1)
- C24 pad 2: +3V3 -> GND
- C24 pad 1: +3V3 -> +2V5
- C24 pad 1: +3V3 -> Net-(C7-Pad1)
- C24 pad 1: VCC -> +3V3
- C24 pad 1: Net-(C19-Pad1) -> +3V3
- C24 pad 1: BOOT0 -> +2V5
- C24 pad 2: Net-(U2-CC) -> GND
- C24 pad 1: Net-(C53-Pad1) -> OSC_IN
- C24 pad 1: NRST -> STM_RST
- C27 pad 2: BOOT0 -> GND
- C28 pad 1: BOOT0 -> GND
- C29 pad 1: BOOT0 -> GND
- C30 pad 2: BOOT0 -> GND
- C35 pad 2: BOOT0 -> GND
- C36 pad 1: BOOT0 -> GND
- C37 pad 1: /FPGA_CLK1 -> 40MHz_OSC
- C37 pad 2: BOOT0 -> GND
- C38 pad 1: BOOT0 -> GND
- C39 pad 1: 40MHz_OSC -> GND
- C39 pad 2: BOOT0 -> CCLK
- C4 pad 1: BOOT0 -> GND
- C40 pad 1: BOOT0 -> GND
- C40 pad 2: uC_CNTRL2 -> uC_CNTRL4
- C41 pad 1: BOOT0 -> GND
- C41 pad 2: uC_CNTRL4 -> +3V3
- C42 pad 1: uC_CNTRL2 -> GND
- C42 pad 2: BOOT0 -> +3V3
- C5 pad 1: BOOT0 -> GND
- C50 pad 1: Net-(U4-VCAP_2) -> GND
- C50 pad 2: BOOT0 -> +3V3
- C52 pad 1: OSC_IN -> GND
- C52 pad 2: BOOT0 -> +3V3
- C6 pad 1: +3V3 -> VCC
- C6 pad 2: BOOT0 -> GND
- IC1 pad 101: BOOT0 -> GND
- IC1 pad 114: BOOT0 -> GND
- IC1 pad 117: BOOT0 -> GND
- IC1 pad 122: uC_CNTRL2 -> CCLK
- IC1 pad 136: BOOT0 -> GND
- IC1 pad 139: BOOT0 -> GND
- IC1 pad 143: Net-(IC1-PROG_B) -> FPGA_CNTRL1
- IC1 pad 16: BOOT0 -> GND
- IC1 pad 22: BOOT0 -> GND
- IC1 pad 29: BOOT0 -> GND
- IC1 pad 37: +2V5 -> Net-(IC1-M1)
- IC1 pad 38: BOOT0 -> Net-(IC1-M0)
- IC1 pad 39: +2V5 -> Net-(IC1-M2)
- IC1 pad 42: BOOT0 -> GND
- IC1 pad 45: BOOT0 -> GND
- IC1 pad 52: unconnected-(IC1-IO_L32P_5/GCLK2-Pad52) -> Net-(IC1-IO_L32P_5/GCLK2)
- IC1 pad 55: Net-(IC1-IO_L32P_4/GCLK0) -> 40MHz_OSC
- IC1 pad 56: 40MHz_OSC -> Net-(IC1-IO_L32N_4/GCLK1)
- IC1 pad 58: Net-(IC1-IO_L31N_4/INIT_B) -> INIT_B
- IC1 pad 64: BOOT0 -> GND
- IC1 pad 67: BOOT0 -> GND
- IC1 pad 71: FPGA_CNTRL3 -> DONE
- IC1 pad 72: Net-(IC1-CCLK) -> CCLK
- IC1 pad 81: BOOT0 -> GND
- IC1 pad 88: BOOT0 -> GND
- IC1 pad 9: BOOT0 -> GND
- IC1 pad 94: BOOT0 -> GND
- IC2 pad 12: BOOT0 -> GND
- IC3 pad 12: BOOT0 -> GND
- IC4 pad 12: BOOT0 -> GND
- IC5 pad 12: BOOT0 -> GND
- J1 pad 1: Net-(J1-Pin_1) -> FPGA_CNTRL1
- J1 pad 2: Net-(J1-Pin_2) -> GND
- J1 pad 3: Net-(J1-Pin_3) -> (no net)
- J1 pad 4: Net-(IC1-TDO) -> (no net)
- J1 pad 5: BOOT0 -> (no net)
- J1 pad 6: BOOT0 -> (no net)
- J1 pad 7: BOOT0 -> (no net)
- J1 pad 8: +3V3 -> (no net)
- J2 pad 1: +3V3 -> Net-(IC1-M2)
- J2 pad 2: SERIAL_RX -> Net-(IC1-M0)
- J2 pad 3: uC_MISO -> Net-(IC1-M1)
- J2 pad 4: uC_SCK -> GND
- J2 pad 5: BOOT0 -> GND
- J2 pad 6: SERIAL_TX -> GND
- J2 pad 7: NRST -> (no net)
- J2 pad 8: uC_MOSI -> (no net)
- J3 pad 2: BOOT0 -> SERIAL_RX
- J3 pad 3: SWIDO -> uC_MISO
- J3 pad 4: BOOT0 -> uC_SCK
- J3 pad 5: unconnected-(J3-Pin_5-Pad5) -> GND
- J3 pad 6: SWCLK -> SERIAL_TX
- J4 pad 1: BOOT0 -> +3V3
- J4 pad 10: unconnected-(J4-A11-Pad10) -> (no net)
- J4 pad 11: unconnected-(J4-A9-Pad11) -> (no net)
- J4 pad 12: unconnected-(J4-A8-Pad12) -> (no net)
- J4 pad 13: unconnected-(J4-A13-Pad13) -> (no net)
- J4 pad 14: unconnected-(J4-A14-Pad14) -> (no net)
- J4 pad 15: WE# -> (no net)
- J4 pad 16: IREQ# -> (no net)
- J4 pad 17: VCC -> (no net)
- J4 pad 18: VCC -> (no net)
- J4 pad 19: MIVAL -> (no net)
- J4 pad 2: D3 -> STM_RST
- J4 pad 20: MCLKI -> (no net)
- J4 pad 21: unconnected-(J4-A12-Pad21) -> (no net)
- J4 pad 22: A7 -> (no net)
- J4 pad 23: A6 -> (no net)
- J4 pad 24: A5 -> (no net)
- J4 pad 25: A4 -> (no net)
- J4 pad 26: A3 -> (no net)
- J4 pad 27: A2 -> (no net)
- J4 pad 28: A1 -> (no net)
- J4 pad 29: A0 -> (no net)
- J4 pad 3: D4 -> JTDO/TRACESWO
- J4 pad 30: D0 -> (no net)
- J4 pad 31: D1 -> (no net)
- J4 pad 32: D2 -> (no net)
- J4 pad 33: unconnected-(J4-IOIS16#-Pad33) -> (no net)
- J4 pad 34: BOOT0 -> (no net)
- J4 pad 35: BOOT0 -> (no net)
- J4 pad 36: Net-(J4-CD1#) -> (no net)
- J4 pad 37: MDO3 -> (no net)
- J4 pad 38: MDO4 -> (no net)
- J4 pad 39: MDO5 -> (no net)
- J4 pad 4: D5 -> GND
- J4 pad 40: MDO6 -> (no net)
- J4 pad 41: MDO7 -> (no net)
- J4 pad 42: unconnected-(J4-CE2#-Pad42) -> (no net)
- J4 pad 43: unconnected-(J4-VS1#/Refresh-Pad43) -> (no net)
- J4 pad 44: IORD# -> (no net)
- J4 pad 45: IOWR# -> (no net)
- J4 pad 46: MISTRT -> (no net)
- J4 pad 47: MDI0 -> (no net)
- J4 pad 48: MDI1 -> (no net)
- J4 pad 49: MDI2 -> (no net)
- J4 pad 5: D6 -> JTMS/SWDIO
- J4 pad 50: MDI3 -> (no net)
- J4 pad 51: VCC -> (no net)
- J4 pad 52: VCC -> (no net)
- J4 pad 53: MDI4 -> (no net)
- J4 pad 54: MDI5 -> (no net)
- J4 pad 55: MDI6 -> (no net)
- J4 pad 56: MDI7 -> (no net)
- J4 pad 57: MCLKO -> (no net)
- J4 pad 58: RESET -> (no net)
- J4 pad 59: unconnected-(J4-WAIT#-Pad59) -> (no net)
- J4 pad 6: D7 -> JTCK/SWCLK
- J4 pad 60: INPACK# -> (no net)
- J4 pad 61: REG# -> (no net)
- J4 pad 62: MOVAL -> (no net)
- J4 pad 63: MOSTRT -> (no net)
- J4 pad 64: MDO0 -> (no net)
- J4 pad 65: MDO1 -> (no net)
- J4 pad 66: MDO2 -> (no net)
- J4 pad 67: Net-(J4-CD2#) -> (no net)
- J4 pad 68: BOOT0 -> (no net)
- J4 pad 7: CE1# -> (no net)
- J4 pad 8: unconnected-(J4-A10-Pad8) -> (no net)
- J4 pad 9: OE# -> (no net)
- R10 pad 1: Net-(IC1-IO_L32P_4/GCLK0) -> _MCLKI
- R10 pad 2: /FPGA_CLK1 -> Net-(IC1-IO_L32P_5/GCLK2)
- R11 pad 1: +3V3 -> STM_RSS_OUT
- R11 pad 2: Net-(IC1-IO_L31N_4/INIT_B) -> Net-(IC1-IO_L32N_4/GCLK1)
- R12 pad 1: Net-(J1-Pin_2) -> +3V3
- R12 pad 2: Net-(IC1-TMS) -> INIT_B
- R15 pad 1: uC_CNTRL2 -> +2V5
- R15 pad 2: Net-(IC1-CCLK) -> DONE
- R17 pad 1: NRST -> STM_RST
- R18 pad 1: Net-(J4-CD1#) -> Net-(J5-CD1#)
- R18 pad 2: BOOT0 -> GND
- R19 pad 1: BOOT0 -> Net-(U5-BOOT0)
- R19 pad 2: Net-(J4-CD2#) -> GND
- R2 pad 1: BOOT0 -> GND
- R20 pad 1: OSC_OUT -> GND
- R20 pad 2: Net-(C53-Pad1) -> Net-(J5-CD2#)
- R21 pad 1: Net-(U4-BOOT0) -> Net-(U5-PA8)
- R21 pad 2: BOOT0 -> STM_RSS_OUT
- R22 pad 1: Net-(J1-Pin_3) -> Net-(JTAG1-Pin_2)
- R22 pad 2: Net-(IC1-TCK) -> Net-(IC1-TMS)
- R22 pad 1: TDI -> Net-(JTAG1-Pin_1)
- R22 pad 2: Net-(J1-Pin_1) -> TDI
- R22 pad 1: +2V5 -> Net-(JTAG1-Pin_3)
- R22 pad 2: FPGA_CNTRL3 -> Net-(IC1-TCK)
- R3 pad 2: Net-(C19-Pad1) -> Net-(C7-Pad1)
- R4 pad 1: BOOT0 -> GND
- R7 pad 1: BOOT0 -> GND
- R8 pad 1: BOOT0 -> GND
- R9 pad 1: FPGA_CNTRL1 -> +2V5
- R9 pad 2: Net-(IC1-PROG_B) -> FPGA_CNTRL1
- RN2 pad 1: unconnected-(RN2-R1.1-Pad1) -> INOUT_A0
- RN2 pad 10: IOWR# -> D2
- RN2 pad 11: IORD# -> MDO1
- RN2 pad 12: OE# -> D1
- RN2 pad 13: MDO7 -> MDO0
- RN2 pad 14: CE1# -> D0
- RN2 pad 15: MDO6 -> MOSTRT
- RN2 pad 16: unconnected-(RN2-R1.2-Pad16) -> A0
- RN2 pad 2: INOUT_MDO6 -> INOUT_MOSTRT
- RN2 pad 3: INOUT_CE1# -> INOUT_D0
- RN2 pad 4: INOUT_MDO7 -> INOUT_MDO0
- RN2 pad 5: INOUT_OE# -> INOUT_D1
- RN2 pad 6: INOUT_IORD# -> INOUT_MDO1
- RN2 pad 7: INOUT_IOWR# -> INOUT_D2
- RN2 pad 8: INOUT_MISTRT -> INOUT_MDO2
- RN2 pad 9: MISTRT -> MDO2
- RN3 pad 1: INOUT_A0 -> unconnected-(RN3-R1.1-Pad1)
- RN3 pad 10: D2 -> IOWR#
- RN3 pad 11: MDO1 -> IORD#
- RN3 pad 12: D1 -> OE#
- RN3 pad 13: MDO0 -> MDO7
- RN3 pad 14: D0 -> CE1#
- RN3 pad 15: MOSTRT -> MDO6
- RN3 pad 16: A0 -> unconnected-(RN3-R1.2-Pad16)
- RN3 pad 2: INOUT_MOSTRT -> INOUT_MDO6
- RN3 pad 3: INOUT_D0 -> INOUT_CE1#
- RN3 pad 4: INOUT_MDO0 -> INOUT_MDO7
- RN3 pad 5: INOUT_D1 -> INOUT_OE#
- RN3 pad 6: INOUT_MDO1 -> INOUT_IORD#
- RN3 pad 7: INOUT_D2 -> INOUT_IOWR#
- RN3 pad 8: INOUT_MDO2 -> INOUT_MISTRT
- RN3 pad 9: MDO2 -> MISTRT
- RN4 pad 12: IREQ# -> unconnected-(RN4-R5.2-Pad12)
- RN4 pad 5: INOUT_IREQ# -> unconnected-(RN4-R5.1-Pad5)
- U1 pad 2: BOOT0 -> GND
- U2 pad 3: BOOT0 -> GND
- U3 pad 11: BOOT0 -> GND
- U3 pad 2: BOOT0 -> GND
- U3 pad 3: BOOT0 -> GND
- U3 pad 5: BOOT0 -> GND
- U4 pad 1: +3V3 -> uC_AD0
- U4 pad 10: uC_MISO -> DONE
- U4 pad 11: uC_MOSI -> GND
- U4 pad 12: BOOT0 -> unconnected-(U4-(DNC)_2-Pad12)
- U4 pad 13: +3V3 -> unconnected-(U4-~CEO-Pad13)
- U4 pad 14: FPGA_CNTRL1 -> unconnected-(U4-(DNC)_6-Pad14)
- U4 pad 16: SERIAL_TX -> unconnected-(U4-(DNC)-Pad16)
- U4 pad 17: SERIAL_RX -> Net-(JTAG1-Pin_4)
- U4 pad 18: BOOT0 -> +3V3
- U4 pad 2: uC_A14 -> unconnected-(U4-(DNC)_3-Pad2)
- U4 pad 20: FPGA_CNTRL2 -> +3V3
- U4 pad 21: FPGA_CNTRL3 -> (no net)
- U4 pad 22: uC_CNTRL1 -> (no net)
- U4 pad 23: uC_CNTRL2 -> (no net)
- U4 pad 24: uC_AD3 -> (no net)
- U4 pad 25: uC_AD4 -> (no net)
- U4 pad 26: unconnected-(U4-PB0-Pad26) -> (no net)
- U4 pad 27: unconnected-(U4-PB1-Pad27) -> (no net)
- U4 pad 28: uC_A9 -> (no net)
- U4 pad 29: uC_SCK -> (no net)
- U4 pad 3: uC_A13 -> CCLK
- U4 pad 30: unconnected-(U4-PB11-Pad30) -> (no net)
- U4 pad 31: Net-(U4-VCAP_1) -> (no net)
- U4 pad 32: +3V3 -> (no net)
- U4 pad 33: unconnected-(U4-PB12-Pad33) -> (no net)
- U4 pad 34: unconnected-(U4-PB13-Pad34) -> (no net)
- U4 pad 35: unconnected-(U4-PB14-Pad35) -> (no net)
- U4 pad 36: unconnected-(U4-PB15-Pad36) -> (no net)
- U4 pad 37: uC_AD5 -> (no net)
- U4 pad 38: uC_AD6 -> (no net)
- U4 pad 39: uC_AD7 -> (no net)
- U4 pad 4: uC_A12 -> Net-(IC1-TDO)
- U4 pad 40: uC_A8 -> (no net)
- U4 pad 41: uC_A15 -> (no net)
- U4 pad 42: uC_A19 -> (no net)
- U4 pad 43: INOUT_IREQ# -> (no net)
- U4 pad 44: unconnected-(U4-PA11-Pad44) -> (no net)
- U4 pad 45: unconnected-(U4-PA12-Pad45) -> (no net)
- U4 pad 46: SWIDO -> (no net)
- U4 pad 47: Net-(U4-VCAP_2) -> (no net)
- U4 pad 48: +3V3 -> (no net)
- U4 pad 49: SWCLK -> (no net)
- U4 pad 5: OSC_IN -> Net-(IC1-TMS)
- U4 pad 50: unconnected-(U4-PA15-Pad50) -> (no net)
- U4 pad 51: unconnected-(U4-PC10-Pad51) -> (no net)
- U4 pad 52: uC_A11 -> (no net)
- U4 pad 53: uC_A10 -> (no net)
- U4 pad 54: uC_AD2 -> (no net)
- U4 pad 55: uC_A16 -> (no net)
- U4 pad 56: uC_CNTRL4 -> (no net)
- U4 pad 57: uC_A17 -> (no net)
- U4 pad 58: unconnected-(U4-PB6-Pad58) -> (no net)
- U4 pad 59: unconnected-(U4-PB7-Pad59) -> (no net)
- U4 pad 6: OSC_OUT -> Net-(IC1-TCK)
- U4 pad 60: Net-(U4-BOOT0) -> (no net)
- U4 pad 61: uC_A18 -> (no net)
- U4 pad 62: uC_CNTRL3 -> (no net)
- U4 pad 63: BOOT0 -> (no net)
- U4 pad 64: +3V3 -> (no net)
- U4 pad 7: NRST -> FPGA_CNTRL1
- U4 pad 8: uC_AD0 -> INIT_B
- U4 pad 9: uC_AD1 -> unconnected-(U4-(DNC)_5-Pad9)
- U5 pad 1: uC_A16 -> +3V3
- U5 pad 10: uC_PROG2 -> uC_MISO
- U5 pad 11: uC_CNTRL1 -> uC_MOSI
- U5 pad 12: +3V3 -> GND
- U5 pad 13: unconnected-(U5-NC-Pad13) -> +3V3
- U5 pad 14: +3V3 -> FPGA_CNTRL1
- U5 pad 16: uC_A19 -> SERIAL_TX
- U5 pad 17: uC_A18 -> SERIAL_RX
- U5 pad 18: uC_A8 -> GND
- U5 pad 19: uC_A7 -> +3V3
- U5 pad 2: uC_A15 -> unconnected-(U5-PC13-Pad2)
- U5 pad 20: uC_A6 -> FPGA_CNTRL2
- U5 pad 21: uC_A5 -> DONE
- U5 pad 22: uC_A4 -> uC_CNTRL1
- U5 pad 23: uC_A3 -> CCLK
- U5 pad 24: uC_A2 -> uC_AD3
- U5 pad 25: uC_A1 -> uC_AD4
- U5 pad 26: uC_CNTRL3 -> unconnected-(U5-PB0-Pad26)
- U5 pad 27: BOOT0 -> unconnected-(U5-PB1-Pad27)
- U5 pad 28: uC_CNTRL2 -> unconnected-(U5-PB2-Pad28)
- U5 pad 29: uC_AD0 -> uC_SCK
- U5 pad 3: uC_A14 -> unconnected-(U5-PC14-Pad3)
- U5 pad 31: uC_AD1 -> Net-(U5-VCAP_1)
- U5 pad 32: unconnected-(U5-DQ9-Pad32) -> +3V3
- U5 pad 33: uC_AD2 -> unconnected-(U5-PB12-Pad33)
- U5 pad 35: uC_AD3 -> unconnected-(U5-PB14-Pad35)
- U5 pad 37: +3V3 -> uC_AD5
- U5 pad 38: uC_AD4 -> uC_AD6
- U5 pad 39: unconnected-(U5-DQ12-Pad39) -> uC_AD7
- U5 pad 4: uC_A13 -> unconnected-(U5-PC15-Pad4)
- U5 pad 40: uC_AD5 -> unconnected-(U5-PC9-Pad40)
- U5 pad 41: unconnected-(U5-DQ13-Pad41) -> Net-(U5-PA8)
- U5 pad 42: uC_AD6 -> _RESET
- U5 pad 43: unconnected-(U5-DQ14-Pad43) -> IREQ#
- U5 pad 44: uC_AD7 -> unconnected-(U5-PA11-Pad44)
- U5 pad 45: uC_A0 -> unconnected-(U5-PA12-Pad45)
- U5 pad 46: BOOT0 -> JTMS/SWDIO
- U5 pad 47: BOOT0 -> Net-(U5-VCAP_2)
- U5 pad 48: uC_A17 -> +3V3
- U5 pad 5: uC_A12 -> OSC_IN
- U5 pad 6: uC_A11 -> OSC_OUT
- U5 pad 7: uC_A10 -> STM_RST
- U5 pad 8: uC_A9 -> uC_AD0
- U5 pad 9: uC_PROG1 -> uC_AD1
- U6 pad 1: BOOT0 -> FLASH_CS
- U6 pad 10: BOOT0 -> (no net)
- U6 pad 11: uC_CNTRL4 -> (no net)
- U6 pad 12: uC_A4 -> (no net)
- U6 pad 13: uC_AD4 -> (no net)
- U6 pad 14: uC_AD5 -> (no net)
- U6 pad 15: uC_A5 -> (no net)
- U6 pad 16: uC_A6 -> (no net)
- U6 pad 17: uC_AD6 -> (no net)
- U6 pad 18: uC_AD7 -> (no net)
- U6 pad 19: uC_A7 -> (no net)
- U6 pad 2: uC_A3 -> FLASH_MOSI
- U6 pad 20: +3V3 -> (no net)
- U6 pad 3: uC_AD3 -> +3V3
- U6 pad 4: uC_AD2 -> GND
- U6 pad 5: uC_A2 -> FLASH_MISO
- U6 pad 6: uC_A1 -> FLASH_SCK
- U6 pad 7: uC_AD1 -> +3V3
- U6 pad 8: uC_AD0 -> +3V3
- U6 pad 9: uC_A0 -> (no net)
- Y1 pad 2: BOOT0 -> GND
- Y1 pad 3: Net-(C19-Pad1) -> Net-(C7-Pad1)
- Y1 pad 4: BOOT0 -> GND
- Y2 pad 2: BOOT0 -> GND
- Y2 pad 3: Net-(C53-Pad1) -> Net-(C55-Pad1)
- Y2 pad 4: BOOT0 -> GND
Routing:
- added copper zone on F.Cu, net uC_SCK
- removed copper zone on F.Cu, net BOOT0
