File: CAM_XILINX_STM/com_1300/com_1300.kicad_sch (KiCad schematic)
At the start: 128 parts, among them J1 Conn_02x20_Counter_Clockwise, J2 9-68RD-0.635SF, J3 MEC1-108-01-S-D-RA1-SL, J4 Conn_02x10_Top_Bottom, U1 LT1963AxST-3.3, U17 MT48LC16M16A2TG-7E, U2 STM32F415RGTx, U3 AM29LV320DT90EC, U4 TC74LCX373FT, U6 LP3982IMM-ADJ, U7 LTC3411EMS, Y1 16mHz, Y2 40mHZ

Commit message: 010424
Parts:
- removed C24: C-OPEN, Capacitor_SMD:C_0603_1608Metric, symbol Device:C_Small
- removed J1: Conn_02x20_Counter_Clockwise, Connector_PinSocket_2.00mm:PinSocket_2x20_P2.00mm_Horizontal, symbol Connector_Generic:Conn_02x20_Odd_Even
- R16, R17: value R-OPEN -> 0
Connections:
- net FPGA_CLK1: no longer U.D5 (IO_VREF_0)
- net GND: no longer R17.1
- net PC_CARD_41: no longer J2.49 (PC_CARD_41), RN4.15 (R2.2)
- net PC_CARD_42: no longer J2.50 (PC_CARD_42), RN4.13 (R4.2)
- net PC_CARD_55: no longer J2.16 (PC_CARD_55), RN4.14 (R3.2)
- net VCC: now also J2.18 (VPP1), J2.52 (VPP2)
- net MCLKO: now reaches U.B8 (IO_L32N_0/GCLK7)
- net MCLKO: now also R17.1
- net BOOT0: no longer names the net of U2.60 (BOOT0)
- net BOOT0: no longer R3.1
- net BOOT_SECTOR: no longer names the net of U2.15 (PA1)
- net CAN2_RX: no longer names the net of U2.59 (PB7)
- net CAN2_RX: no longer J4.5 (Pin_5)
- net CAN2_TX: no longer names the net of U2.58 (PB6)
- net CAN2_TX: no longer J4.7 (Pin_7)
- net GPIO_1: no longer names the net of U2.50 (PA15)
- net GPIO_1: no longer J4.11 (Pin_11)
- net PC_CARD_1 renamed D3
- net PC_CARD_10 renamed A9
- net PC_CARD_11 renamed A8
- net PC_CARD_12 renamed A13
- net PC_CARD_13 renamed A14
- net PC_CARD_14 renamed WE#
- net PC_CARD_15 renamed MIVAL
- net PC_CARD_16 renamed MCLKI
- net PC_CARD_17 renamed A12
- net PC_CARD_18 renamed A7
- net PC_CARD_19 renamed A6
- net PC_CARD_2 renamed D4
- net PC_CARD_20 renamed A5
- net PC_CARD_21 renamed A4
- net PC_CARD_22 renamed A3
- net PC_CARD_23 renamed A2
- net PC_CARD_24 renamed A1
- net PC_CARD_25 renamed A0
- net PC_CARD_26 renamed D0
- net PC_CARD_27 renamed D1
- net PC_CARD_28 renamed D2
- net PC_CARD_29 renamed IOIS16#
- net PC_CARD_3 renamed D5
- net PC_CARD_30 renamed MDO3
- net PC_CARD_31 renamed MDO4
- net PC_CARD_32 renamed MDO5
- net PC_CARD_33 renamed MDO6
- net PC_CARD_34 renamed MDO7
- net PC_CARD_35 renamed CE2#
- net PC_CARD_36 renamed IORD#
- net PC_CARD_37 renamed IOWR#
- net PC_CARD_38 renamed MISTRT
- net PC_CARD_39 renamed MDI0
- net PC_CARD_4 renamed D6
- net PC_CARD_40 renamed MDI1
- net PC_CARD_43 renamed MDI4
- net PC_CARD_44 renamed MDI5
- net PC_CARD_45 renamed MDI6
- net PC_CARD_46 renamed MDI7
- net PC_CARD_47 renamed WAIT#
- net PC_CARD_48 renamed INPACK#
- net PC_CARD_49 renamed REG#
- net PC_CARD_5 renamed D7
- net PC_CARD_50 renamed MOVAL
- net PC_CARD_51 renamed MOSTRT
- net PC_CARD_52 renamed MDO0
- net PC_CARD_53 renamed MDO1
- net PC_CARD_54 renamed MDO2
- net PC_CARD_6 renamed CE1#
- net PC_CARD_7 renamed A10
- net PC_CARD_8 renamed OE#
- net PC_CARD_9 renamed A11
- net PC_CARD_RESET renamed RESET
- net SERIAL_IO_1: no longer names the net of U.A4 (IO_L01P_0/VRN_0)
- net SERIAL_IO_2: no longer names the net of U.C5 (IO_L25N_0)
- net SPI2_MISO: no longer names the net of U2.35 (PB14)
- net SPI2_MISO: no longer J4.8 (Pin_8)
- net SPI2_MOSI: no longer names the net of U2.36 (PB15)
- net SPI2_MOSI: no longer J4.10 (Pin_10)
- net SPI2_SCK: no longer names the net of U2.34 (PB13)
- net SPI2_SCK: no longer J4.6 (Pin_6)
- net SWCLK: no longer names the net of U2.49 (PA14)
- net SWCLK: no longer J4.13 (Pin_13)
- net SWIDO: no longer names the net of U2.46 (PA13)
- net SWIDO: no longer R9.2
- net TIM3_CH3: no longer names the net of U2.26 (PB0)
- net TIM3_CH3: no longer J4.3 (Pin_3)
- net TIM3_CH4: no longer names the net of U2.27 (PB1)
- net TIM3_CH4: no longer J4.1 (Pin_1)
- net USART3_CK: no longer names the net of U2.33 (PB12)
- net USART3_CK: no longer J4.4 (Pin_4)
- net USART3_RX: no longer names the net of U2.30 (PB11)
- net USART3_RX: no longer J4.2 (Pin_2)
- net USART3_TX: no longer names the net of U2.51 (PC10)
- net USART3_TX: no longer J4.9 (Pin_9)
- net USB_D+: no longer names the net of U2.45 (PA12)
- net USB_D+: no longer J4.14 (Pin_14)
- net USB_D-: no longer names the net of U2.44 (PA11)
- net USB_D-: no longer J4.12 (Pin_12)
- net USER_IO_0: no longer names the net of U.G2 (IO)
- net USER_IO_1: no longer names the net of U.C1 (IO_L01N_7/VRP_7)
- net USER_IO_10: no longer names the net of U.E2 (IO_L20P_7)
- net USER_IO_11: no longer names the net of U.F4 (IO_L21N_7)
- net USER_IO_12: no longer names the net of U.E4 (IO_L21P_7)
- net USER_IO_13: no longer names the net of U.F2 (IO_L22N_7)
- net USER_IO_14: no longer names the net of U.F3 (IO_L22P_7)
- net USER_IO_15: no longer names the net of U.G5 (IO_L23N_7)
- net USER_IO_16: no longer names the net of U.F5 (IO_L23P_7)
- net USER_IO_17: no longer names the net of U.G3 (IO_L24N_7)
- net USER_IO_18: no longer names the net of U.G4 (IO_L24P_7)
- net USER_IO_19: no longer names the net of U.H3 (IO_L39N_7)
- net USER_IO_2: no longer names the net of U.B1 (IO_L01P_7/VRN_7)
- net USER_IO_20: no longer names the net of U.H4 (IO_L39P_7)
- net USER_IO_21: no longer names the net of U.A9 (IO)
- net USER_IO_22: no longer names the net of U.A12 (IO)
- net USER_IO_23: no longer names the net of U.C10 (IO)
- net USER_IO_24: no longer names the net of U.D12 (IO/VREF_1)
- net USER_IO_25: no longer names the net of U.A14 (IO_L01N_1/VRP_1)
- net USER_IO_26: no longer names the net of U.B14 (IO_L01P_1/VRN_1)
- net USER_IO_27: no longer names the net of U.A13 (IO_L10N_1/VREF_1)
- net USER_IO_28: no longer names the net of U.B13 (IO_L10P_1)
- net USER_IO_29: no longer names the net of U.B12 (IO_L27N_1)
- net USER_IO_3: no longer names the net of U.C2 (IO_L16N_7)
- net USER_IO_30: no longer names the net of U.C12 (IO_L27P_1)
- net USER_IO_31: no longer names the net of U.D11 (IO_L28N_1)
- net USER_IO_4: no longer names the net of U.C3 (IO_L16P_7/VREF_7)
- net USER_IO_5: no longer names the net of U.D1 (IO_L17N_7)
- net USER_IO_6: no longer names the net of U.D2 (IO_L17P_7)
- net USER_IO_7: no longer names the net of U.E3 (IO_L19N_7/VREF_7)
- net USER_IO_8: no longer names the net of U.D3 (IO_L19P_7)
- net USER_IO_9: no longer names the net of U.E1 (IO_L20N_7)
- new net IREQ#: J2.16 (IREQ#), RN4.14 (R3.2)
- new net MDI2: J2.49 (MDI2), RN4.15 (R2.2)
- new net MDI3: J2.50 (MDI3), RN4.13 (R4.2)
- no-connect marks 14 -> 66
Other:
- note removed: "40 Pin Connector"
- moved on the sheet: C24, R4, U3, Y2

Commit message: 010424
Parts:
- removed RN8: 8 x 10K, Resistor_SMD:R_Cat16-8, symbol Device:R_Pack08
- added C24: C-OPEN, Capacitor_SMD:C_0603_1608Metric, symbol Device:C_Small
- added R18: 4.7K, Resistor_SMD:R_0402_1005Metric, symbol Device:R_Small
- added R20: 56, Resistor_SMD:R_0402_1005Metric, symbol Device:R_Small
- added R22: 56, Resistor_SMD:R_0603_1608Metric, symbol Device:R_Small
- added TP3, TP4: TestPoint_Small, TestPoint:TestPoint_Pad_D1.0mm, symbol Connector:TestPoint_Small
- added U9: XC3S400-PQ208, symbol FPGA_Xilinx:XC3S400-PQ208
- R17: value 0 -> 330
Connections:
- net +1V2: now also U9.174 (VCCINT), U9.192 (VCCINT), U9.70 (VCCINT), U9.88 (VCCINT)
- net +2V5: now also R17.1, U9.121 (VCCAUX), U9.142 (VCCAUX), U9.17 (VCCAUX), U9.173 (VCCAUX), U9.193 (VCCAUX), U9.38 (VCCAUX), U9.54 (M1), U9.56 (M2), U9.69 (VCCAUX), U9.89 (VCCAUX)
- net +3V3: now also R18.1, U9.110 (VCCO_3), U9.127 (VCCO_3), U9.136 (VCCO_2), U9.153 (VCCO_2), U9.164 (VCCO_1), U9.177 (VCCO_1), U9.188 (VCCO_0), U9.201 (VCCO_0), U9.23 (VCCO_7), U9.32 (VCCO_6), U9.49 (VCCO_6), U9.6 (VCCO_7), U9.60 (VCCO_5), U9.73 (VCCO_5), U9.84 (VCCO_4), U9.98 (VCCO_4)
- net FPGA_CNTRL1: now also R22.1
- net FPGA_CNTRL3: now also R17.2, TP3.1, U9.103 (DONE)
- net GND: now also C24.2, U9.1 (GND), U9.105 (GND), U9.112 (GND), U9.118 (GND), U9.129 (GND), U9.134 (GND), U9.14 (GND), U9.145 (GND), U9.151 (GND), U9.157 (GND), U9.163 (GND), U9.170 (GND), U9.179 (GND), U9.186 (GND), U9.195 (GND), U9.202 (GND), U9.25 (GND), U9.30 (GND), U9.41 (GND), U9.47 (GND), U9.53 (GND), U9.55 (M0), U9.59 (GND), U9.66 (GND), U9.75 (GND), U9.8 (GND), U9.82 (GND), U9.91 (GND), U9.99 (GND)
- net MCLKO: now also J2.57 (MCLKO), RN6.13 (R4.2); no longer R17.1, U.B8 (IO_L32N_0/GCLK7)
- net SDRAM_A0: now also U9.132 (IO_L40P_2/VREF_2)
- net SDRAM_A1: now also U9.131 (IO_L40N_3/VREF_3)
- net SDRAM_A10: now also U9.119 (IO_L22P_3)
- net SDRAM_A11: now also U9.117 (IO_L21N_3)
- net SDRAM_A12: now also U9.116 (IO_L21P_3)
- net SDRAM_A2: now also U9.130 (IO_L40P_3)
- net SDRAM_A3: now also U9.128 (IO_L39N_3)
- net SDRAM_A4: now also U9.126 (IO_L39P_3)
- net SDRAM_A5: now also U9.125 (IO_L24N_3)
- net SDRAM_A6: now also U9.124 (IO_L24P_3)
- net SDRAM_A7: now also U9.123 (IO_L23N_3)
- net SDRAM_A8: now also U9.122 (IO_L23P_3/VREF_3)
- net SDRAM_A9: now also U9.120 (IO_L22N_3)
- net SDRAM_CNTRL10: now also U9.144 (IO_L22N_2)
- net SDRAM_CNTRL2: now also U9.155 (IO_L01P_2/VRN_2)
- net SDRAM_CNTRL3: now also U9.154 (IO/VREF_2)
- net SDRAM_CNTRL4: now also U9.152 (IO_L19N_2)
- net SDRAM_CNTRL5: now also U9.150 (IO_L19P_2)
- net SDRAM_CNTRL6: now also U9.149 (IO_L20N_2)
- net SDRAM_CNTRL7: now also U9.148 (IO_L20P_2)
- net SDRAM_CNTRL8: now also U9.147 (IO-L21N_2)
- net SDRAM_CNTRL9: now also U9.146 (IO_L21P_2)
- net SDRAM_DQ0: now also U9.115 (IO_L20N_3)
- net SDRAM_DQ1: now also U9.114 (IO_L20P_3)
- net SDRAM_DQ10: now also U9.137 (IO_L39N_2)
- net SDRAM_DQ11: now also U9.138 (IO_L24P_2)
- net SDRAM_DQ12: now also U9.139 (IO_L24N_2)
- net SDRAM_DQ13: now also U9.140 (IO_L23P_2)
- net SDRAM_DQ14: now also U9.141 (IO_L23N_2/VREF_2)
- net SDRAM_DQ15: now also U9.143 (IO_L22P_2)
- net SDRAM_DQ2: now also U9.113 (IO_L19N_3)
- net SDRAM_DQ3: now also U9.111 (IO_L19P_3)
- net SDRAM_DQ4: now also U9.109 (IO_L17N_3)
- net SDRAM_DQ5: now also U9.108 (IO_L17P_3/VREF_3)
- net SDRAM_DQ6: now also U9.107 (IO_L01N_3/VRP_3)
- net SDRAM_DQ7: now also U9.106 (IO_L01P_3/VRN_3)
- net SDRAM_DQ8: now also U9.133 (IO_L40N_2)
- net SDRAM_DQ9: now also U9.135 (IO_L39P_2)
- net uC_CNTRL2: now also C24.1, R20.1
- net at J2.36 (CD1#), R16.1: no longer J2.43 (VS1#/Refresh)
- net A10: no longer names the net of J2.8 (A10)
- net A10: no longer RN6.13 (R4.2)
- net A11: no longer names the net of RN6.10 (R7.2)
- net A11: no longer J2.10 (A11)
- net A12: no longer names the net of RN3.16 (R1.2)
- net A12: no longer J2.21 (A12)
- net A13: no longer names the net of RN5.12 (R5.2)
- net A13: no longer J2.13 (A13)
- net A14: no longer names the net of RN5.10 (R7.2)
- net A14: no longer J2.14 (A14)
- net A8: no longer names the net of RN5.14 (R3.2)
- net A8: no longer J2.12 (A8)
- net A9: no longer names the net of RN5.16 (R1.2)
- net A9: no longer J2.11 (A9)
- net CE2#: no longer names the net of RN6.12 (R5.2)
- net CE2#: no longer J2.42 (CE2#)
- net INOUT_PC_CARD_10: no longer names the net of RN5.1 (R1.1)
- net INOUT_PC_CARD_10: no longer U.T10 (IO/VREF_4)
- net INOUT_PC_CARD_11: no longer names the net of RN5.3 (R3.1)
- net INOUT_PC_CARD_11: no longer U.R13 (IO_L01N_4/VRP_4)
- net INOUT_PC_CARD_12: no longer names the net of RN5.5 (R5.1)
- net INOUT_PC_CARD_12: no longer U.T13 (IO_L01P_4/VRN_4)
- net INOUT_PC_CARD_13: no longer names the net of RN5.7 (R7.1)
- net INOUT_PC_CARD_13: no longer U.P12 (IO_L25N_4)
- net INOUT_PC_CARD_17: no longer names the net of RN3.1 (R1.1)
- net INOUT_PC_CARD_17: no longer U.R11 (IO_L28P_4)
- net INOUT_PC_CARD_26 renamed INOUT_D0
- net INOUT_PC_CARD_27 renamed INOUT_D1
- net INOUT_PC_CARD_28 renamed INOUT_D2
- net INOUT_PC_CARD_29: no longer names the net of U.T5 (IO)
- net INOUT_PC_CARD_29: no longer RN1.8 (R8.1)
- net INOUT_PC_CARD_35: no longer names the net of U.J4 (IO_L39N_6)
- net INOUT_PC_CARD_35: no longer RN6.5 (R5.1)
- net INOUT_PC_CARD_47: no longer names the net of RN2.1 (R1.1)
- net INOUT_PC_CARD_47: no longer U.M4 (IO_L19N_6)
- net INOUT_PC_CARD_7: no longer names the net of U.T14 (IO)
- net INOUT_PC_CARD_7: no longer RN6.4 (R4.1)
- net INOUT_PC_CARD_9: no longer names the net of U.P13 (IO/VREF_4)
- net INOUT_PC_CARD_9: no longer RN6.7 (R7.1)
- net IOIS16#: no longer names the net of J2.33 (IOIS16#)
- net IOIS16#: no longer RN1.9 (R8.2)
- net WAIT#: no longer names the net of RN2.16 (R1.2)
- net WAIT#: no longer J2.59 (WAIT#)
- new net: R22.2, U9.207 (PROG_B)
- new net: R20.2, U9.104 (CCLK)
- new net: R18.2, TP4.1
- new net INOUT_MCLKO: RN6.4 (R4.1), U.B8 (IO_L32N_0/GCLK7)
- no-connect marks 66 -> 75
Other:
- moved on the sheet: R16

Commit message: 020424
Parts:
- removed C24: C-OPEN, Capacitor_SMD:C_0603_1608Metric, symbol Device:C_Small
- removed R17: 330, Resistor_SMD:R_0402_1005Metric, symbol Device:R_Small
- removed R18: 4.7K, Resistor_SMD:R_0402_1005Metric, symbol Device:R_Small
- removed R20: 56, Resistor_SMD:R_0402_1005Metric, symbol Device:R_Small
- removed R22: 56, Resistor_SMD:R_0603_1608Metric, symbol Device:R_Small
- removed TP3, TP4: TestPoint_Small, TestPoint:TestPoint_Pad_D1.0mm, symbol Connector:TestPoint_Small
- removed U9: XC3S400-PQ208, symbol FPGA_Xilinx:XC3S400-PQ208
Connections:
- net INOUT_PC_CARD_2 is gone; now on net INOUT_D2: RN7.2 (R2.1), U.J14 (IO_L39N_3)
- net INOUT_PC_CARD_55: no longer RN4.3 (R3.1), U.G1 (IO_L40P_7)
- net INOUT_PC_CARD_1 renamed INOUT_D3
- net INOUT_PC_CARD_14 renamed INOUT_WE#
- net INOUT_PC_CARD_15 renamed INOUT_MIVAL
- net INOUT_PC_CARD_16 renamed INOUT_MCLKI
- net INOUT_PC_CARD_18 renamed INOUT_A7
- net INOUT_PC_CARD_19 renamed INOUT_A6
- net INOUT_PC_CARD_20 renamed INOUT_A5
- net INOUT_PC_CARD_21 renamed INOUT_A4
- net INOUT_PC_CARD_22 renamed INOUT_A3
- net INOUT_PC_CARD_23 renamed INOUT_A2
- net INOUT_PC_CARD_24 renamed INOUT_A1
- net INOUT_PC_CARD_25 renamed INOUT_A0
- net INOUT_PC_CARD_3 renamed INOUT_D5
- net INOUT_PC_CARD_30 renamed INOUT_MDO3
- net INOUT_PC_CARD_31 renamed INOUT_MDO4
- net INOUT_PC_CARD_32 renamed INOUT_MDO5
- net INOUT_PC_CARD_33 renamed INOUT_MDO6
- net INOUT_PC_CARD_34 renamed INOUT_MDO7
- net INOUT_PC_CARD_36 renamed INOUT_IORD#
- net INOUT_PC_CARD_37 renamed INOUT_IOWR#
- net INOUT_PC_CARD_38 renamed INOUT_MISTRT
- net INOUT_PC_CARD_39 renamed INOUT_MDI0
- net INOUT_PC_CARD_4 renamed INOUT_D6
- net INOUT_PC_CARD_40 renamed INOUT_MDI1
- net INOUT_PC_CARD_41 renamed INOUT_MDI2
- net INOUT_PC_CARD_42 renamed INOUT_MDI3
- net INOUT_PC_CARD_43 renamed INOUT_MDI4
- net INOUT_PC_CARD_44 renamed INOUT_MDI5
- net INOUT_PC_CARD_45 renamed INOUT_MDI6
- net INOUT_PC_CARD_46 renamed INOUT_MDI7
- net INOUT_PC_CARD_48 renamed INOUT_INPACK#
- net INOUT_PC_CARD_49 renamed INOUT_REG#
- net INOUT_PC_CARD_5 renamed INOUT_D7
- net INOUT_PC_CARD_50 renamed INOUT_MOVAL
- net INOUT_PC_CARD_51 renamed INOUT_MOSTRT
- net INOUT_PC_CARD_52 renamed INOUT_MDO0
- net INOUT_PC_CARD_53 renamed INOUT_MDO1
- net INOUT_PC_CARD_54 renamed INOUT_MDO2
- net INOUT_PC_CARD_6 renamed INOUT_CE1#
- net INOUT_PC_CARD_8 renamed INOUT_OE#
- net INOUT_PC_CARD_RESET renamed INOUT_RESET
- new net INOUT_IREQ#: RN4.3 (R3.1), U.G1 (IO_L40P_7)

Commit message: 22323
Parts:
- removed C24 (x8): C-OPEN, Capacitor_SMD:C_0603_1608Metric, symbol Device:C_Small
- removed U17: MT48LC16M16A2TG-7E, Package_SO:TSOP-II-54_22.2x10.16mm_P0.8mm, symbol Storage:MT48LC16M16A2TG-7E
Connections:
- net INOUT_D2: no longer U.J14 (IO_L39N_3)
- net INOUT_D3: no longer U.K13 (IO_L24P_3)
- net INOUT_D5: no longer U.J13 (IO_L39P_3)
- net INOUT_D6: no longer U.J16 (IO_L40N_3/VREF_3)
- net INOUT_D7: no longer U.K16 (IO_L40P_3)
- net SDRAM_A0: no longer names the net of U.C16 (IO_L01P_2/VRN_2)
- net SDRAM_A1: no longer names the net of U.C15 (IO_L16N_2)
- net SDRAM_A10: no longer names the net of U.F13 (IO_L21P_2)
- net SDRAM_A11: no longer names the net of U.F14 (IO_L22N_2)
- net SDRAM_A12: no longer names the net of U.F15 (IO_L22P_2)
- net SDRAM_A2: no longer names the net of U.D14 (IO_L16P_2)
- net SDRAM_A3: no longer names the net of U.D15 (IO_L17N_2)
- net SDRAM_A4: no longer names the net of U.D16 (IO_L17P_2/VREF_2)
- net SDRAM_A5: no longer names the net of U.E13 (IO_L19N_2)
- net SDRAM_A6: no longer names the net of U.E14 (IO_L19P_2)
- net SDRAM_A7: no longer names the net of U.E15 (IO_L20N_2)
- net SDRAM_A8: no longer names the net of U.E16 (IO_L20P_2)
- net SDRAM_A9: no longer names the net of U.F12 (IO_L21N_2)
- net SDRAM_CNTRL1: no longer names the net of U.K14 (IO_L24N_3)
- net SDRAM_CNTRL10: no longer names the net of U.N14 (IO_L19P_3)
- net SDRAM_CNTRL2: no longer names the net of U.L12 (IO_L23P_3/VREF_3)
- net SDRAM_CNTRL3: no longer names the net of U.K12 (IO_L23N_3)
- net SDRAM_CNTRL4: no longer names the net of U.L14 (IO_L22P_3)
- net SDRAM_CNTRL5: no longer names the net of U.L15 (IO_L22N_3)
- net SDRAM_CNTRL6: no longer names the net of U.M13 (IO_L21P_3)
- net SDRAM_CNTRL7: no longer names the net of U.L13 (IO_L21N_3)
- net SDRAM_CNTRL8: no longer names the net of U.M15 (IO_L20P_3)
- net SDRAM_CNTRL9: no longer names the net of U.M16 (IO_L20N_3)
- net SDRAM_DQ0: no longer names the net of U.G12 (IO_L23N_2/VREF_2)
- net SDRAM_DQ1: no longer names the net of U.G13 (IO_L23P_2)
- net SDRAM_DQ10: no longer names the net of U.R16 (IO_L01P_3/VRN_3)
- net SDRAM_DQ11: no longer names the net of U.P15 (IO_L16N_3)
- net SDRAM_DQ12: no longer names the net of U.P14 (IO_L16P_3)
- net SDRAM_DQ13: no longer names the net of U.N16 (IO_L17N_3)
- net SDRAM_DQ14: no longer names the net of U.N15 (IO_L17P_3/VREF_3)
- net SDRAM_DQ15: no longer names the net of U.M14 (IO_L19N_3)
- net SDRAM_DQ2: no longer names the net of U.G14 (IO_L24N_2)
- net SDRAM_DQ3: no longer names the net of U.G15 (IO_L24P_2)
- net SDRAM_DQ4: no longer names the net of U.H13 (IO_L39N_2)
- net SDRAM_DQ5: no longer names the net of U.H14 (IO_L39P_2)
- net SDRAM_DQ6: no longer names the net of U.H15 (IO_L40N_2)
- net SDRAM_DQ7: no longer names the net of U.H16 (IO_L40P_2/VREF_2)
- net SDRAM_DQ8: no longer names the net of U.K15 (IO)
- net SDRAM_DQ9: no longer names the net of U.P16 (IO_L01N_3/VRP_3)
Other:
- note removed: "SDRAM"

Commit message: 124214
Parts:
- removed J4: Conn_02x10_Top_Bottom, Connector_PinHeader_1.27mm:PinHeader_2x08_P1.27mm_Vertical_SMD, symbol Connector_Generic:Conn_02x08_Top_Bottom
- removed R3: 10K, Resistor_SMD:R_0402_1005Metric, symbol Device:R_Small
- removed R9: 0, Resistor_SMD:R_0402_1005Metric, symbol Device:R_Small
- renumbered C16 to C33, C25 to C35, C23 to C36, C22 to C37, C4 to C39, C9 to C49, C12 to C50, C8 to C51, C18 to C52, C2 to C53, C19 to C54, C1 to C55, C20 to C56, C10 to C57, C17 to C58, C15 to C59, C14 to C60, C27 to C61, C26 to C62, J3 to J1, R12 to R1, R5 to R10, R7 to R11, R23 to R12, R10 to R13, R6 to R14, R16 to R15, R15 to R16, R1 to R17, R4 to R2, R2 to R3, R14 to R4, R11 to R5, R13 to R6, R8 to R7, R21 to R9, RN3 to RN2, RN5 to RN3, RN7 to RN4, RN2 to RN5, RN4 to RN6, RN6 to RN7, U6 to U2, U7 to U3, U2 to U5, U3 to U6, U4 to U7, Y2 to Y1, Y1 to Y2
Connections:
- no-connect marks 75 -> 129
Other:
- note removed: "STM free pins"
