File: CAM_XILINX_STM/com_1300/com_1300.kicad_sch (KiCad schematic)
At the start: 112 parts, among them J1 MEC1-108-01-S-D-RA1-SL, J2 9-68RD-0.635SF, U1 LT1963AxST-3.3, U2 LP3982IMM-ADJ, U3 LTC3411EMS, U5 STM32F415RGTx, U6 AM29LV320DT90EC, U7 TC74LCX373FT, Y1 40mHZ, Y2 16mHz

Commit message: 234
Other:
- moved on the sheet: C62

Commit message: 2342342
Parts:
- removed C49, C50, C51, C62: C-OPEN, Capacitor_SMD:C_0402_1005Metric, symbol Device:C_Small
- removed R4: 330, Resistor_SMD:R_0402_1005Metric, symbol Device:R_Small
- removed R5: 4.7K, Resistor_SMD:R_0402_1005Metric, symbol Device:R_Small
- removed R9: 56, Resistor_SMD:R_0402_1005Metric, symbol Device:R_Small
- removed U: XC3S400-4FT256C, Package_BGA:Xilinx_FTG256, symbol FPGA_Xilinx:XC3S400-4FT256C
- added C57, C58, C59, C60: C-OPEN, Capacitor_SMD:C_0402_1005Metric, symbol Device:C_Small
- added IC1: XC3S400-4TQ144C, QFP50P2200X2200X160-144N, symbol XC3S400-4TQ144C:XC3S400-4TQ144C
- added J2: Conn_02x10_Top_Bottom, Connector_PinHeader_1.27mm:PinHeader_2x08_P1.27mm_Vertical_SMD, symbol Connector_Generic:Conn_02x08_Top_Bottom
- added R10: 0, Resistor_SMD:R_0201_0603Metric, symbol Device:R_Small
- added R11: 4.7K, Resistor_SMD:R_0402_1005Metric, symbol Device:R_Small
- added R12: 330, Resistor_SMD:R_0402_1005Metric, symbol Device:R_Small
- R13: value 0 -> 56; footprint Resistor_SMD:R_0201_0603Metric -> Resistor_SMD:R_0402_1005Metric
- renumbered C39 to C38, C52 to C48, C53 to C49, C54 to C50, C55 to C51, C56 to C52, C57 to C53, C58 to C54, C59 to C55, C60 to C56, J2 to J3, R6 to R4, R7 to R5, R10 to R6, R11 to R7, R12 to R8, U5 to U4, U6 to U5, U7 to U6
Connections:
- net INOUT_PC_CARD_55 is gone; now on net INOUT_IREQ#: U4.43 (PA10)
- net +1V2: now also IC1.121 (VCCINT_3), IC1.133 (VCCINT_4), IC1.49 (VCCINT_1), IC1.61 (VCCINT_2)
- net +2V5: now also IC1.120 (VCCAUX_3), IC1.134 (VCCAUX_4), IC1.37 (M1), IC1.39 (M2), IC1.48 (VCCAUX_1), IC1.62 (VCCAUX_2), R12.1
- net +3V3: now also IC1.106 (VCCO_RIGHT_3), IC1.115 (VCCO_TOP_1), IC1.126 (VCCO_TOP_2), IC1.138 (VCCO_TOP_3), IC1.19 (VCCO_LEFT_2), IC1.3 (VCCO_LEFT_1), IC1.34 (VCCO_LEFT_3), IC1.43 (VCCO_BOTTOM_1), IC1.54 (VCCO_BOTTOM_2), IC1.66 (VCCO_BOTTOM_3), IC1.75 (VCCO_RIGHT_1), IC1.91 (VCCO_RIGHT_2), R11.1
- net 40MHz_OSC: now also C59.1, IC1.56 (IO_L32N_4/GCLK1)
- net FPGA_CLK1: now also C57.1, R10.2; no longer C61.1, R13.2
- net FPGA_CNTRL2: now also IC1.40 (IO_L01P_5/CS_B), IC1.41 (IO__L01N_5/RDWR_B)
- net FPGA_CNTRL3: now also TP2.1, IC1.71 (DONE), R12.2; no longer TP1.1
- net FPGA_TEST_EDGE1: now also IC1.137 (IO_L27N_0)
- net FPGA_TEST_EDGE2: now also IC1.135 (IO_L27P_0)
- net FPGA_TEST_EDGE3: now also IC1.132 (IO_L30N_0)
- net FPGA_TEST_EDGE4: now also IC1.131 (IO_L30P_0)
- net FPGA_TEST_EDGE5: now also IC1.130 (IO_L31N_0)
- net FPGA_TEST_EDGE6: now also IC1.129 (IO_L31P_0/VREF_0)
- net GND: now also C61.1, C57.2, C58.1, C59.2, C60.1, IC1.101 (GND_12), IC1.114 (GND_13), IC1.117 (GND_14), IC1.136 (GND_15), IC1.139 (GND_16), IC1.16 (GND_2), IC1.22 (GND_3), IC1.29 (GND_4), IC1.38 (M0), IC1.42 (GND_5), IC1.45 (GND_6), IC1.64 (GND_7), IC1.67 (GND_8), IC1.81 (GND_9), IC1.88 (GND_10), IC1.9 (GND_1), IC1.94 (GND_11); no longer C61.2
- net INOUT_A0: now also IC1.15 (IO_L24N_7)
- net INOUT_A1: now also IC1.14 (IO_L24P_7)
- net INOUT_A2: now also IC1.13 (IO_L23N_7)
- net INOUT_A3: now also IC1.12 (IO_L23P_7)
- net INOUT_A4: now also IC1.11 (IO_L22N_7)
- net INOUT_A5: now also IC1.10 (IO_L22P_7)
- net INOUT_A6: now also IC1.8 (IO_L21N_7)
- net INOUT_A7: now also IC1.7 (IO_L21P_7)
- net INOUT_CE1#: now also IC1.90 (IO_L40N_3/VREF_3)
- net INOUT_D0: now also IC1.78 (IO_L20N_3)
- net INOUT_D1: now also IC1.79 (IO_L21P_3)
- net INOUT_D2: now also IC1.80 (IO_L21N_3); no longer RN4.2 (R2.1)
- net INOUT_D3: now also IC1.82 (IO_L22P_3)
- net INOUT_D5: now also IC1.84 (IO_L23P_3/VREF_3)
- net INOUT_D6: now also IC1.85 (IO_L23N_3)
- net INOUT_D7: now also IC1.86 (IO_L24P_3)
- net INOUT_INPACK#: now also IC1.20 (IO_L40P_6/VREF_6)
- net INOUT_IORD#: now also IC1.95 (IO_L24P_2)
- net INOUT_IOWR#: now also IC1.93 (IO_L40N_2)
- net INOUT_IREQ#: now also IC1.77 (IO_L20P_3)
- net INOUT_MCLKI: now also IC1.108 (IO_L01N_2/VRP_2), IC1.53 (IO_L32N_5/GCLK3)
- net INOUT_MCLKO: now also RN2.1 (R1.1), IC1.6 (IO_L20N_7); no longer RN7.4 (R4.1)
- net INOUT_MDI0: now also IC1.96 (IO_L24N_2)
- net INOUT_MDI1: now also IC1.97 (IO_L23P_2)
- net INOUT_MDI2: now also IC1.98 (IO_L23N_2/VREF_2)
- net INOUT_MDI3: now also IC1.99 (IO_L22P_2)
- net INOUT_MDI4: now also IC1.100 (IO_L22N_2)
- net INOUT_MDI5: now also IC1.102 (IO_L21P_2)
- net INOUT_MDI6: now also IC1.103 (IO_L21N_2)
- net INOUT_MDI7: now also IC1.104 (IO_L20P_2)
- net INOUT_MDO0: now also IC1.33 (IO_L20N_6)
- net INOUT_MDO1: now also IC1.32 (IO_L20P_6)
- net INOUT_MDO2: now also IC1.31 (IO_L21N_6)
- net INOUT_MDO3: now also IC1.30 (IO_L21P_6)
- net INOUT_MDO4: now also IC1.28 (IO_L22N_6)
- net INOUT_MDO5: now also IC1.27 (IO_L22P_6)
- net INOUT_MDO6: now also IC1.26 (IO_L23N_6)
- net INOUT_MDO7: now also IC1.25 (IO_L23P_6)
- net INOUT_MISTRT: now also IC1.92 (IO_L40P_2/VREF_2)
- net INOUT_MIVAL: now also IC1.24 (IO_L24N_6/VREF_6)
- net INOUT_MOSTRT: now also IC1.87 (IO_L24N_3)
- net INOUT_MOVAL: now also IC1.23 (IO_L24P_6)
- net INOUT_OE#: now also IC1.89 (IO_L40P_3)
- net INOUT_REG#: now also IC1.21 (IO_L40N_6)
- net INOUT_RESET: now also IC1.105 (IO_L20N_2)
- net INOUT_WE#: now also IC1.107 (IO_L01P_2/VRN_2)
- net MCLKO: now also RN2.16 (R1.2); no longer RN7.13 (R4.2)
- net uC_AD0: now also IC1.65 (IO_L27N_4/DIN/D0)
- net uC_AD1: now also IC1.63 (O_L27P_4/D1)
- net uC_AD2: now also IC1.60 (IO_L30N_4/D2)
- net uC_AD3: now also IC1.59 (IO_L30P_4/D3)
- net uC_AD4: now also IC1.51 (IO_L31N_5/D4)
- net uC_AD5: now also IC1.50 (IO_L31P_5/D5)
- net uC_AD6: now also IC1.47 (IO_L28N_5/D6)
- net uC_AD7: now also IC1.46 (IO_L28P_5/D7)
- net uC_CNTRL1: now also C58.2, IC1.123 (IO_L31N_1/VREF_1)
- net uC_CNTRL2: now also R13.1, C60.2, IC1.122 (IO_L31P_1)
- net uC_CNTRL3: now also IC1.119 (IO_L28N_1)
- net uC_CNTRL4: now also C61.2, IC1.118 (IO_L28P_1)
- net at R22.2: now also IC1.143 (PROG_B)
- new net: IC1.55 (IO_L32P_4/GCLK0), R10.1
- new net: IC1.58 (IO_L31N_4/INIT_B), R11.2, TP1.1
- new net: IC1.72 (CCLK), R13.2
- new net INOUT_D4: IC1.83 (IO_L22N_3), RN4.2 (R2.1)
- no-connect marks 129 -> 40

Commit message: 23623637
Parts:
- removed C24 (x20): C-OPEN, Capacitor_SMD:C_0603_1608Metric, symbol Device:C_Small
- removed J2: Conn_02x10_Top_Bottom, Connector_PinHeader_1.27mm:PinHeader_2x08_P1.27mm_Vertical_SMD, symbol Connector_Generic:Conn_02x08_Top_Bottom
- added J1: Conn_02x04_Top_Bottom, Connector_PinHeader_1.27mm:PinHeader_2x04_P1.27mm_Vertical, symbol Connector_Generic:Conn_02x04_Top_Bottom
- added R22 (x3): 56, Resistor_SMD:R_0603_1608Metric, symbol Device:R_Small
- renumbered C33 to C1, C38 to C18, C48 to C24, C49 to C25, C50 to C26, C51 to C27, C52 to C28, C53 to C29, C35 to C3, C54 to C30, C55 to C35, C56 to C36, C57 to C37, C58 to C38, C59 to C39, C36 to C4, C60 to C40, C61 to C41, C37 to C5, J1 to J2, R12 to R14, R13 to R15, R14 to R17, R15 to R18, R16 to R19, R17 to R20
Connections:
- net +3V3: now also J1.1 (Pin_1)
- net GND: now also J1.5 (Pin_5)
- net at IC1.109 (TDO): now also J1.4 (Pin_4)
- net at IC1.110 (TCK): now also R22.2
- net at IC1.111 (TMS): now also R22.2
- net TDI: now reaches IC1.144 (TDI)
- net TDI: now also R22.1
- new net: J1.3 (Pin_3), R22.1
- new net: J1.2 (Pin_2), R22.1
- new net: J1.6 (Pin_6), R22.2
Other:
- moved on the sheet: C24, C37, C38, C39, C40, C41, IC1, R10, R11, R14, R15, R22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

Commit message: 2234545
Parts:
- removed J2: MEC1-108-01-S-D-RA1-SL, Connector_PinSocket_1.27mm:PinSocket_2x08_P1.27mm_Vertical_SMD, symbol Connector:MEC1-108-01-S-D-RA1-SL
- removed RN7: 8 x 180R, Resistor_SMD:R_Cat16-8, symbol Device:R_Pack08
- added J2: Conn_02x04_Top_Bottom, Connector_PinHeader_1.27mm:PinHeader_2x04_P1.27mm_Vertical, symbol Connector_Generic:Conn_02x04_Top_Bottom
- renumbered C3 to C2, R3 to R2, R2 to R3, RN2 to RN1, RN3 to RN2, RN1 to RN3, RN6 to RN4, RN4 to RN5, RN5 to RN6
Connections:
- net FPGA_TEST_EDGE1 is gone; now on net INOUT_WE#: IC1.137 (IO_L27N_0)
- net FPGA_TEST_EDGE2 is gone; now on net INOUT_RESET: IC1.135 (IO_L27P_0)
- net FPGA_TEST_EDGE3 is gone; now on net INOUT_IORD#: IC1.132 (IO_L30N_0)
- net FPGA_TEST_EDGE4 is gone; now on net INOUT_IOWR#: IC1.131 (IO_L30P_0)
- net FPGA_TEST_EDGE5 is gone; now on net INOUT_MISTRT: IC1.130 (IO_L31N_0)
- net +3V3: now also J1.8 (Pin_8), J2.1 (Pin_1); no longer J1.1 (Pin_1)
- net A0: now also RN3.16 (R1.2); no longer RN6.9 (R8.2)
- net A1: now also RN6.10 (R7.2); no longer RN6.11 (R6.2)
- net A2: now also RN6.12 (R5.2); no longer RN6.13 (R4.2)
- net A3: now also RN6.14 (R3.2); no longer RN6.15 (R2.2)
- net A4: now also RN6.15 (R2.2); no longer RN1.9 (R8.2)
- net A5: now also RN1.9 (R8.2); no longer RN1.11 (R6.2)
- net A6: now also RN1.11 (R6.2); no longer RN1.12 (R5.2)
- net A7: now also RN1.13 (R4.2); no longer RN1.14 (R3.2)
- net CE1#: now also RN2.14 (R3.2)
- net D0: now also RN3.14 (R3.2); no longer RN3.15 (R2.2)
- net D1: now also RN3.12 (R5.2); no longer RN3.13 (R4.2)
- net D2: now also RN3.10 (R7.2); no longer RN3.11 (R6.2)
- net GND: now also J1.6 (Pin_6), J1.7 (Pin_7), J2.5 (Pin_5)
- net INOUT_A0: now also IC1.14 (IO_L24P_7), RN3.1 (R1.1); no longer IC1.15 (IO_L24N_7), RN6.8 (R8.1)
- net INOUT_A1: now also IC1.13 (IO_L23N_7), RN6.7 (R7.1); no longer IC1.14 (IO_L24P_7), RN6.6 (R6.1)
- net INOUT_A2: now also IC1.12 (IO_L23P_7), RN6.5 (R5.1); no longer IC1.13 (IO_L23N_7), RN6.4 (R4.1)
- net INOUT_A3: now also IC1.11 (IO_L22N_7), RN6.3 (R3.1); no longer IC1.12 (IO_L23P_7), RN6.2 (R2.1)
- net INOUT_A4: now also IC1.10 (IO_L22P_7), RN6.2 (R2.1); no longer IC1.11 (IO_L22N_7), RN1.8 (R8.1)
- net INOUT_A5: now also IC1.8 (IO_L21N_7), RN1.8 (R8.1); no longer IC1.10 (IO_L22P_7), RN1.6 (R6.1)
- net INOUT_A6: now also IC1.7 (IO_L21P_7), RN1.6 (R6.1); no longer IC1.8 (IO_L21N_7), RN1.5 (R5.1)
- net INOUT_A7: now also IC1.6 (IO_L20N_7), RN1.4 (R4.1); no longer IC1.7 (IO_L21P_7), RN1.3 (R3.1)
- net INOUT_CE1#: now also IC1.93 (IO_L40N_2), RN2.3 (R3.1); no longer IC1.90 (IO_L40N_3/VREF_3)
- net INOUT_D0: now also IC1.77 (IO_L20P_3), RN3.3 (R3.1); no longer IC1.78 (IO_L20N_3), RN3.2 (R2.1)
- net INOUT_D1: now also IC1.78 (IO_L20N_3), RN3.5 (R5.1); no longer IC1.79 (IO_L21P_3), RN3.4 (R4.1)
- net INOUT_D2: now also IC1.79 (IO_L21P_3), RN3.7 (R7.1); no longer IC1.80 (IO_L21N_3), RN3.6 (R6.1)
- net INOUT_D3: now also IC1.80 (IO_L21N_3); no longer IC1.82 (IO_L22P_3)
- net INOUT_D4: now also IC1.82 (IO_L22P_3); no longer IC1.83 (IO_L22N_3)
- net INOUT_D5: now also IC1.83 (IO_L22N_3); no longer IC1.84 (IO_L23P_3/VREF_3)
- net INOUT_INPACK#: now also IC1.15 (IO_L24N_7), RN6.4 (R4.1); no longer IC1.20 (IO_L40P_6/VREF_6), RN6.3 (R3.1)
- net INOUT_IORD#: now also RN2.6 (R6.1); no longer IC1.95 (IO_L24P_2)
- net INOUT_IOWR#: now also RN2.7 (R7.1); no longer IC1.93 (IO_L40N_2), RN2.2 (R2.1)
- net INOUT_IREQ#: now also IC1.33 (IO_L20N_6), RN4.5 (R5.1); no longer IC1.77 (IO_L20P_3), RN4.3 (R3.1)
- net INOUT_MCLKI: now also IC1.105 (IO_L20N_2), RN1.1 (R1.1); no longer IC1.108 (IO_L01N_2/VRP_2), IC1.53 (IO_L32N_5/GCLK3), RN4.7 (R7.1)
- net INOUT_MCLKO: now also IC1.5 (IO_L20P_7), RN1.7 (R7.1); no longer IC1.6 (IO_L20N_7), RN1.1 (R1.1)
- net INOUT_MDI0: now also IC1.95 (IO_L24P_2), RN4.1 (R1.1); no longer IC1.96 (IO_L24N_2), RN2.6 (R6.1)
- net INOUT_MDI1: now also IC1.96 (IO_L24N_2), RN4.2 (R2.1); no longer IC1.97 (IO_L23P_2), RN2.8 (R8.1)
- net INOUT_MDI2: now also IC1.97 (IO_L23P_2), RN4.4 (R4.1); no longer IC1.98 (IO_L23N_2/VREF_2), RN4.2 (R2.1)
- net INOUT_MDI3: now also RN4.6 (R6.1); no longer RN4.4 (R4.1)
- net INOUT_MDI4: now also RN4.8 (R8.1); no longer RN4.6 (R6.1)
- net INOUT_MDI5: now also RN1.2 (R2.1); no longer RN4.8 (R8.1)
- net INOUT_MDI6: now also RN1.3 (R3.1); no longer RN1.2 (R2.1)
- net INOUT_MDI7: now also RN1.5 (R5.1); no longer RN1.4 (R4.1)
- net INOUT_MDO0: now also IC1.32 (IO_L20P_6), RN3.4 (R4.1); no longer IC1.33 (IO_L20N_6), RN3.3 (R3.1)
- net INOUT_MDO1: now also IC1.31 (IO_L21N_6), RN3.6 (R6.1); no longer IC1.32 (IO_L20P_6), RN3.5 (R5.1)
- net INOUT_MDO2: now also IC1.30 (IO_L21P_6), RN3.8 (R8.1); no longer IC1.31 (IO_L21N_6), RN3.7 (R7.1)
- net INOUT_MDO3: now also IC1.28 (IO_L22N_6); no longer IC1.30 (IO_L21P_6)
- net INOUT_MDO4: now also IC1.27 (IO_L22P_6); no longer IC1.28 (IO_L22N_6)
- net INOUT_MDO5: now also IC1.26 (IO_L23N_6); no longer IC1.27 (IO_L22P_6)
- net INOUT_MDO6: now also IC1.25 (IO_L23P_6), RN2.2 (R2.1); no longer IC1.26 (IO_L23N_6)
- net INOUT_MDO7: now also IC1.24 (IO_L24N_6/VREF_6), RN2.4 (R4.1); no longer IC1.25 (IO_L23P_6)
- net INOUT_MISTRT: now also RN2.8 (R8.1); no longer IC1.92 (IO_L40P_2/VREF_2), RN2.4 (R4.1)
- net INOUT_MIVAL: now also IC1.23 (IO_L24P_6), RN4.7 (R7.1); no longer IC1.24 (IO_L24N_6/VREF_6), RN4.5 (R5.1)
- net INOUT_MOSTRT: now also RN3.2 (R2.1); no longer RN3.1 (R1.1)
- net INOUT_MOVAL: now also IC1.21 (IO_L40N_6), RN6.8 (R8.1); no longer IC1.23 (IO_L24P_6), RN6.7 (R7.1)
- net INOUT_OE#: now also RN2.5 (R5.1)
- net INOUT_REG#: now also IC1.17 (IO_L40P_7), RN6.6 (R6.1); no longer IC1.21 (IO_L40N_6), RN6.5 (R5.1)
- net INOUT_RESET: now also RN6.1 (R1.1); no longer IC1.105 (IO_L20N_2), RN1.7 (R7.1)
- net INOUT_WE#: now also RN4.3 (R3.1); no longer IC1.107 (IO_L01P_2/VRN_2), RN4.1 (R1.1)
- net INPACK#: now also RN6.13 (R4.2); no longer RN6.14 (R3.2)
- net IORD#: now also RN2.11 (R6.2)
- net IOWR#: now also RN2.10 (R7.2); no longer RN2.15 (R2.2)
- net IREQ#: now also RN4.12 (R5.2); no longer RN4.14 (R3.2)
- net MCLKI: now also RN1.16 (R1.2); no longer RN4.10 (R7.2)
- net MCLKO: now also RN1.10 (R7.2); no longer RN1.16 (R1.2)
- net MDI0: now also RN4.16 (R1.2); no longer RN2.11 (R6.2)
- net MDI1: now also RN4.15 (R2.2); no longer RN2.9 (R8.2)
- net MDI2: now also RN4.13 (R4.2); no longer RN4.15 (R2.2)
- net MDI3: now also RN4.11 (R6.2); no longer RN4.13 (R4.2)
- net MDI4: now also RN4.9 (R8.2); no longer RN4.11 (R6.2)
- net MDI5: now also RN1.15 (R2.2); no longer RN4.9 (R8.2)
- net MDI6: now also RN1.14 (R3.2); no longer RN1.15 (R2.2)
- net MDI7: now also RN1.12 (R5.2); no longer RN1.13 (R4.2)
- net MDO0: now also RN3.13 (R4.2); no longer RN3.14 (R3.2)
- net MDO1: now also RN3.11 (R6.2); no longer RN3.12 (R5.2)
- net MDO2: now also RN3.9 (R8.2); no longer RN3.10 (R7.2)
- net MDO6: now also RN2.15 (R2.2)
- net MDO7: now also RN2.13 (R4.2)
- net MISTRT: now also RN2.9 (R8.2); no longer RN2.13 (R4.2)
- net MIVAL: now also RN4.10 (R7.2); no longer RN4.12 (R5.2)
- net MOSTRT: now also RN3.15 (R2.2); no longer RN3.16 (R1.2)
- net MOVAL: now also RN6.9 (R8.2); no longer RN6.10 (R7.2)
- net NRST: now also J2.7 (Pin_7)
- net OE#: now also RN2.12 (R5.2)
- net REG#: now also RN6.11 (R6.2); no longer RN6.12 (R5.2)
- net RESET: now also RN6.16 (R1.2); no longer RN1.10 (R7.2)
- net SERIAL_RX: now also J2.2 (Pin_2)
- net SERIAL_TX: now also J2.6 (Pin_6)
- net WE#: now also RN4.14 (R3.2); no longer RN4.16 (R1.2)
- net uC_PROG1: now also J2.3 (Pin_3)
- net uC_PROG2: now also J2.4 (Pin_4)
- net uC_PROG4: now also J2.8 (Pin_8)
- net at R22.2: now also J1.1 (Pin_1); no longer J1.6 (Pin_6)
- net FPGA_TEST_EDGE6: no longer names the net of IC1.129 (IO_L31P_0/VREF_0)
- no-connect marks 40 -> 38
Other:
- note added: "CI Card Connector"
- note removed: "PC Card Connector"
- moved on the sheet: C24, R3, RN1, RN2, RN4, RN5, RN6, Y1

Commit message: tracert
Parts:
- added J3: Conn_02x03_Top_Bottom, Connector_PinHeader_1.27mm:PinHeader_1x06_P1.27mm_Horizontal, symbol Connector_Generic:Conn_02x03_Top_Bottom
- R18: footprint Resistor_SMD:R_0402_1005Metric -> Resistor_SMD:R_0201_0603Metric
- renumbered J3 to J4
Connections:
- net +3V3: now also J3.1 (Pin_1)
- net GND: now also J3.4 (Pin_4)
- net INOUT_A0: now also IC1.95 (IO_L24P_2); no longer IC1.14 (IO_L24P_7)
- net INOUT_A1: now also IC1.96 (IO_L24N_2); no longer IC1.13 (IO_L23N_7)
- net INOUT_A2: now also IC1.97 (IO_L23P_2); no longer IC1.12 (IO_L23P_7)
- net INOUT_A3: now also IC1.99 (IO_L22P_2); no longer IC1.11 (IO_L22N_7)
- net INOUT_A4: now also IC1.100 (IO_L22N_2); no longer IC1.10 (IO_L22P_7)
- net INOUT_A5: now also IC1.102 (IO_L21P_2); no longer IC1.8 (IO_L21N_7)
- net INOUT_A6: now also IC1.103 (IO_L21N_2); no longer IC1.7 (IO_L21P_7)
- net INOUT_A7: now also IC1.104 (IO_L20P_2); no longer IC1.6 (IO_L20N_7)
- net INOUT_CE1#: now also IC1.15 (IO_L24N_7); no longer IC1.93 (IO_L40N_2)
- net INOUT_D0: now also IC1.31 (IO_L21N_6); no longer IC1.77 (IO_L20P_3)
- net INOUT_D1: now also IC1.30 (IO_L21P_6); no longer IC1.78 (IO_L20N_3)
- net INOUT_D2: now also IC1.28 (IO_L22N_6); no longer IC1.79 (IO_L21P_3)
- net INOUT_D3: now also IC1.27 (IO_L22P_6); no longer IC1.80 (IO_L21N_3)
- net INOUT_D4: now also IC1.26 (IO_L23N_6); no longer IC1.82 (IO_L22P_3)
- net INOUT_D5: now also IC1.25 (IO_L23P_6); no longer IC1.83 (IO_L22N_3)
- net INOUT_D6: now also IC1.24 (IO_L24N_6/VREF_6); no longer IC1.85 (IO_L23N_3)
- net INOUT_D7: now also IC1.23 (IO_L24P_6); no longer IC1.86 (IO_L24P_3)
- net INOUT_INPACK#: now also IC1.93 (IO_L40N_2); no longer IC1.15 (IO_L24N_7)
- net INOUT_IREQ#: now also IC1.32 (IO_L20P_6); no longer IC1.33 (IO_L20N_6)
- net INOUT_MCLKI: now also IC1.5 (IO_L20P_7); no longer IC1.105 (IO_L20N_2)
- net INOUT_MCLKO: now also IC1.105 (IO_L20N_2); no longer IC1.5 (IO_L20P_7)
- net INOUT_MDI0: now also IC1.14 (IO_L24P_7); no longer IC1.95 (IO_L24P_2)
- net INOUT_MDI1: now also IC1.13 (IO_L23N_7); no longer IC1.96 (IO_L24N_2)
- net INOUT_MDI2: now also IC1.12 (IO_L23P_7); no longer IC1.97 (IO_L23P_2)
- net INOUT_MDI3: now also IC1.11 (IO_L22N_7); no longer IC1.99 (IO_L22P_2)
- net INOUT_MDI4: now also IC1.10 (IO_L22P_7); no longer IC1.100 (IO_L22N_2)
- net INOUT_MDI5: now also IC1.8 (IO_L21N_7); no longer IC1.102 (IO_L21P_2)
- net INOUT_MDI6: now also IC1.7 (IO_L21P_7); no longer IC1.103 (IO_L21N_2)
- net INOUT_MDI7: now also IC1.6 (IO_L20N_7); no longer IC1.104 (IO_L20P_2)
- net INOUT_MDO0: now also IC1.76 (IO_1); no longer IC1.32 (IO_L20P_6)
- net INOUT_MDO1: now also IC1.77 (IO_L20P_3); no longer IC1.31 (IO_L21N_6)
- net INOUT_MDO2: now also IC1.78 (IO_L20N_3); no longer IC1.30 (IO_L21P_6)
- net INOUT_MDO3: now also IC1.79 (IO_L21P_3); no longer IC1.28 (IO_L22N_6)
- net INOUT_MDO4: now also IC1.80 (IO_L21N_3); no longer IC1.27 (IO_L22P_6)
- net INOUT_MDO5: now also IC1.82 (IO_L22P_3); no longer IC1.26 (IO_L23N_6)
- net INOUT_MDO6: now also IC1.83 (IO_L22N_3); no longer IC1.25 (IO_L23P_6)
- net INOUT_MDO7: now also IC1.85 (IO_L23N_3); no longer IC1.24 (IO_L24N_6/VREF_6)
- net INOUT_MIVAL: now also IC1.86 (IO_L24P_3); no longer IC1.23 (IO_L24P_6)
- net INOUT_MOSTRT: now also IC1.21 (IO_L40N_6); no longer IC1.87 (IO_L24N_3)
- net INOUT_MOVAL: now also IC1.87 (IO_L24N_3); no longer IC1.21 (IO_L40N_6)
- net INOUT_OE#: now also IC1.17 (IO_L40P_7); no longer IC1.89 (IO_L40P_3)
- net INOUT_REG#: now also IC1.89 (IO_L40P_3); no longer IC1.17 (IO_L40P_7)
- net uC_PROG1: no longer J2.3 (Pin_3), U4.10 (PC2)
- net uC_PROG2: no longer J2.4 (Pin_4), U4.29 (PB10)
- net SWIDO: now reaches U4.46 (PA13)
- net SWIDO: now also J3.3 (Pin_3)
- net SWCLK: now reaches U4.49 (PA14)
- net SWCLK: now also J3.6 (Pin_6)
- net BOOT0: now reaches U4.60 (BOOT0)
- net BOOT0: now also J3.2 (Pin_2)
- net uC_PROG4 renamed uC_MOSI
- new net uC_MISO: J2.3 (Pin_3), U4.10 (PC2)
- new net uC_SCK: J2.4 (Pin_4), U4.29 (PB10)
- no-connect marks 38 -> 35
Other:
- moved on the sheet: R18

Commit message: 123
Parts:
- added C55, C56, C57, C58: 100 nF, Capacitor_SMD:C_0201_0603Metric, symbol Device:C_Small
- added IC2, IC3, IC4: SN74CBTD3384CDBR, SN74CBTD3384CDBR:SOP65P780X200-24N, symbol SN74CBTD3384CDBR:SN74CBTD3384CDBR
- added IC5: SN74CBTD3384CDBR, SOP65P780X200-24N, symbol SN74CBTD3384CDBR:SN74CBTD3384CDBR
- RN1, RN2, RN3, RN4, RN5, RN6: value 8 x 180R -> 8 x 30R
Connections:
- net +3V3: now also C55.2, C56.2, C57.2, C58.2, IC2.24 (VCC), IC3.24 (VCC), IC4.24 (VCC), IC5.24 (VCC)
- net GND: now also C55.1, C56.1, C57.1, C58.1, IC2.12 (GND), IC3.12 (GND), IC4.12 (GND), IC5.12 (GND)
- net INOUT_A0: now also IC2.11 (1A5); no longer IC1.95 (IO_L24P_2)
- net INOUT_A1: now also IC3.22 (2A5); no longer IC1.96 (IO_L24N_2)
- net INOUT_A2: now also IC3.18 (2A3); no longer IC1.97 (IO_L23P_2)
- net INOUT_A3: now also IC3.17 (2A2); no longer IC1.99 (IO_L22P_2)
- net INOUT_A4: now also IC3.14 (2A1); no longer IC1.100 (IO_L22N_2)
- net INOUT_A5: now also IC3.4 (1A2)
- net INOUT_A6: now also IC3.7 (1A3); no longer IC1.103 (IO_L21N_2)
- net INOUT_A7: now also IC3.11 (1A5); no longer IC1.104 (IO_L20P_2)
- net INOUT_CE1#: now also IC5.14 (2A1); no longer IC1.15 (IO_L24N_7)
- net INOUT_D0: now also IC2.7 (1A3); no longer IC1.31 (IO_L21N_6)
- net INOUT_D1: now also IC2.4 (1A2); no longer IC1.30 (IO_L21P_6)
- net INOUT_D2: now also IC2.3 (1A1); no longer IC1.28 (IO_L22N_6)
- net INOUT_D3: now also IC5.11 (1A5); no longer IC1.27 (IO_L22P_6)
- net INOUT_D4: now also IC5.8 (1A4); no longer IC1.26 (IO_L23N_6)
- net INOUT_D5: now also IC5.7 (1A3); no longer IC1.25 (IO_L23P_6)
- net INOUT_D6: now also IC5.4 (1A2); no longer IC1.24 (IO_L24N_6/VREF_6)
- net INOUT_D7: now also IC5.3 (1A1); no longer IC1.23 (IO_L24P_6)
- net INOUT_IORD#: now also IC5.18 (2A3)
- net INOUT_IOWR#: now also IC5.21 (2A4)
- net INOUT_MCLKI: now also IC4.18 (2A3); no longer IC1.5 (IO_L20P_7)
- net INOUT_MDI0: now also IC4.11 (1A5); no longer IC1.14 (IO_L24P_7)
- net INOUT_MDI1: now also IC4.8 (1A4); no longer IC1.13 (IO_L23N_7)
- net INOUT_MDI2: now also IC4.4 (1A2); no longer IC1.12 (IO_L23P_7)
- net INOUT_MDI3: now also IC4.3 (1A1); no longer IC1.11 (IO_L22N_7)
- net INOUT_MDI4: now also IC4.17 (2A2); no longer IC1.10 (IO_L22P_7)
- net INOUT_MDI5: now also IC4.21 (2A4); no longer IC1.8 (IO_L21N_7)
- net INOUT_MDI6: now also IC4.22 (2A5); no longer IC1.7 (IO_L21P_7)
- net INOUT_MDI7: now also IC3.8 (1A4); no longer IC1.6 (IO_L20N_7)
- net INOUT_MISTRT: now also IC5.22 (2A5)
- net INOUT_MIVAL: now also IC4.14 (2A1); no longer IC1.86 (IO_L24P_3)
- net INOUT_OE#: now also IC5.17 (2A2); no longer IC1.17 (IO_L40P_7)
- net INOUT_REG#: now also IC3.21 (2A4); no longer IC1.89 (IO_L40P_3)
- net INOUT_RESET: now also IC3.3 (1A1); no longer IC1.135 (IO_L27P_0)
- net INOUT_WE#: now also IC4.7 (1A3)
- new net BUS_OE: IC2.1 (1~{OE}), IC2.13 (2~{OE}), IC3.1 (1~{OE}), IC3.13 (2~{OE}), IC4.1 (1~{OE}), IC4.13 (2~{OE}), IC5.1 (1~{OE}), IC5.13 (2~{OE})
- new net _A0: IC1.95 (IO_L24P_2), IC2.10 (1B5)
- new net _A1: IC1.96 (IO_L24N_2), IC3.23 (2B5)
- new net _A2: IC1.97 (IO_L23P_2), IC3.19 (2B3)
- new net _A3: IC1.99 (IO_L22P_2), IC3.16 (2B2)
- new net _A4: IC1.100 (IO_L22N_2), IC3.15 (2B1)
- new net _A5: IC3.5 (1B2)
- new net _A6: IC1.103 (IO_L21N_2), IC3.6 (1B3)
- new net _A7: IC1.104 (IO_L20P_2), IC3.10 (1B5)
- new net _CE1#: IC1.15 (IO_L24N_7), IC5.15 (2B1)
- new net _D0: IC1.31 (IO_L21N_6), IC2.6 (1B3)
- new net _D1: IC1.30 (IO_L21P_6), IC2.5 (1B2)
- new net _D2: IC1.28 (IO_L22N_6), IC2.2 (1B1)
- new net _D3: IC1.27 (IO_L22P_6), IC5.10 (1B5)
- new net _D4: IC1.26 (IO_L23N_6), IC5.9 (1B4)
- new net _D5: IC1.25 (IO_L23P_6), IC5.6 (1B3)
- new net _D6: IC1.24 (IO_L24N_6/VREF_6), IC5.5 (1B2)
- new net _D7: IC1.23 (IO_L24P_6), IC5.2 (1B1)
- new net _IORD#: IC5.19 (2B3)
- new net _IOWR#: IC5.20 (2B4)
- new net _MCLKI: IC1.5 (IO_L20P_7), IC4.19 (2B3)
- new net _MDI0: IC1.14 (IO_L24P_7), IC4.10 (1B5)
- new net _MDI1: IC1.13 (IO_L23N_7), IC4.9 (1B4)
- new net _MDI2: IC1.12 (IO_L23P_7), IC4.5 (1B2)
- new net _MDI3: IC1.11 (IO_L22N_7), IC4.2 (1B1)
- new net _MDI4: IC1.10 (IO_L22P_7), IC4.16 (2B2)
- new net _MDI5: IC1.8 (IO_L21N_7), IC4.20 (2B4)
- new net _MDI6: IC1.7 (IO_L21P_7), IC4.23 (2B5)
- new net _MDI7: IC1.6 (IO_L20N_7), IC3.9 (1B4)
- new net _MISTRT: IC5.23 (2B5)
- new net _MIVAL: IC1.86 (IO_L24P_3), IC4.15 (2B1)
- new net _OE#: IC1.17 (IO_L40P_7), IC5.16 (2B2)
- new net _REG#: IC1.89 (IO_L40P_3), IC3.20 (2B4)
- new net _RESET: IC1.135 (IO_L27P_0), IC3.2 (1B1)
- new net _WE#: IC4.6 (1B3)
- no-connect marks 35 -> 47
Other:
- moved on the sheet: C24, J2, J3, J4, R18, R19, RN1, RN2, RN3, RN4, RN5, RN6

Commit message: 566565
Connections:
- net BUS_OE: now also IC1.33 (IO_L20N_6)
- net INOUT_A5: no longer IC1.102 (IO_L21P_2)
- net INOUT_IORD#: no longer IC1.132 (IO_L30N_0)
- net INOUT_IOWR#: no longer IC1.131 (IO_L30P_0)
- net INOUT_MISTRT: no longer IC1.130 (IO_L31N_0)
- net INOUT_WE#: no longer IC1.137 (IO_L27N_0)
- net _A5: now also IC1.102 (IO_L21P_2)
- net _IORD#: now also IC1.132 (IO_L30N_0)
- net _IOWR#: now also IC1.131 (IO_L30P_0)
- net _MISTRT: now also IC1.130 (IO_L31N_0)
- net _WE#: now also IC1.137 (IO_L27N_0)
- no-connect marks 47 -> 81
Other:
- moved on the sheet: C57, IC5, RN1, RN2, RN3
