File: CAM_XILINX_STM/com_1300/com_1300.kicad_sch (KiCad schematic)
At the start: 104 parts, among them IC1 XC3S400-4TQ144C, IC2 SN74CBTD3384CDBR, IC3 SN74CBTD3384CDBR, IC4 SN74CBTD3384CDBR, IC5 SN74CBTD3384CDBR, J1 Conn_02x04_Top_Bottom, J2 Conn_02x04_Top_Bottom, J3 Conn_02x03_Top_Bottom, J4 9-68RD-0.635SF, U1 LT1963AxST-3.3, U2 LP3982IMM-ADJ, U3 LTC3411EMS, U4 STM32F415RGTx, U5 AM29LV320DT90EC, U6 TC74LCX373FT, Y1 40mHZ, Y2 16mHz

Commit message: fdsdsf
Parts:
- C38, C40, C41: value C-OPEN -> 100 nF; footprint Capacitor_SMD:C_0402_1005Metric -> Capacitor_SMD:C_0201_0603Metric
Changed lines of the file:
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@@
       (effects (font (size 1.27 1.27)) (justify left))
     )
-    (property "Value" "C-OPEN" (at 218.948 31.496 90)
+    (property "Value" "100 nF" (at 218.948 31.496 90)
       (effects (font (size 1.27 1.27)) (justify left))
     )
-    (property "Footprint" "Capacitor_SMD:C_0402_1005Metric" (at 217.424 33.274 0)
+    (property "Footprint" "Capacitor_SMD:C_0201_0603Metric" (at 217.424 33.274 0)
       (effects (font (size 1.27 1.27)) hide)
     )
@@
       (effects (font (size 1.27 1.27)) (justify left))
     )
-    (property "Value" "C-OPEN" (at 198.374 34.29 90)
+    (property "Value" "100 nF" (at 198.374 34.29 90)
       (effects (font (size 1.27 1.27)) (justify left))
     )
-    (property "Footprint" "Capacitor_SMD:C_0402_1005Metric" (at 199.644 35.814 0)
+    (property "Footprint" "Capacitor_SMD:C_0201_0603Metric" (at 199.644 35.814 0)
       (effects (font (size 1.27 1.27)) hide)
     )
@@
       (effects (font (size 1.27 1.27)) (justify left))
     )
-    (property "Value" "C-OPEN" (at 203.454 31.496 90)
+    (property "Value" "100 nF" (at 203.454 31.496 90)
       (effects (font (size 1.27 1.27)) (justify left))
     )
-    (property "Footprint" "Capacitor_SMD:C_0402_1005Metric" (at 202.184 32.512 0)
+    (property "Footprint" "Capacitor_SMD:C_0201_0603Metric" (at 202.184 32.512 0)
       (effects (font (size 1.27 1.27)) hide)
     )
