File: CAM_XILINX_STM/com_1300/com_1300.kicad_sch (KiCad schematic)
At the start: 104 parts, among them IC1 XC3S400-4TQ144C, IC2 SN74CBTD3384CDBR, IC3 SN74CBTD3384CDBR, IC4 SN74CBTD3384CDBR, IC5 SN74CBTD3384CDBR, J2 Conn_02x04_Top_Bottom, J3 Conn_02x03_Top_Bottom, J4 9-68RD-0.635SF, J5 Conn_02x03_Top_Bottom, J8 Conn_01x02, U1 LT1963AxST-3.3, U2 LP3982IMM-ADJ, U3 LTC3411EMS, U4 STM32F415RGTx, U7 W25Q64BVSSIG, U9 XCF02SVOG20C, Y1 40mHZ, Y2 16mHz

Commit message: 32244
Parts:
- renumbered C24 to C20, C25 to C21, C26 to C22, C39 to C37, C40 to C39, C41 to C40, C55 to C41, C58 to C42, C56 to C50, C57 to C52, C18 to C6, J8 to J1, J5 to J2, J2 to J3, J3 to J4, J4 to J5, JTAG to JTAG1, R24 to R11, R11 to R12, R14 to R15, R21 to R19, R19 to R20, R15 to R21, R20 to R22, R26 to R9, RN3 to RN2, RN2 to RN3, U9 to U4, U4 to U5, U7 to U6
Connections:
- net VCC: no longer J5.18 (VPP1), J5.52 (VPP2)
- no-connect marks 73 -> 75
