File: CAM_XILINX_STM/com_1300/_autosave-com_1300.kicad_pcb (KiCad board)
At the start: 4 copper layers, 50 x 75.9 mm, 112 parts, among them J1 MEC1-108-01-S-D-RA1-SL, J2 9-68RD-0.635SF, U1 LT1963AxST-3.3, U2 LP3982IMM-ADJ, U3 LTC3411EMS, U5 STM32F415RGTx, U6 AM29LV320DT90EC, U7 TC74LCX373FT, Y1 40mHZ, Y2 16mHz

Commit message: 234543
Routing:
- net VCC: track 8.12 -> 86.4 mm, vias 0 -> 2
- net FPGA_CNTRL3: track 0.00 -> 70.4 mm, vias 0 -> 5
- net uC_A14: track 0.00 -> 66.8 mm, vias 0 -> 2
- net uC_CNTRL2: track 18.3 -> 69.4 mm, vias 1 -> 3
- net +2V5: track 75.6 -> 120.1 mm, vias 0 -> 3
- net /FPGA_CLK1: track 0.00 -> 43.9 mm, vias 0 -> 2
- net INOUT_CE1#: track 0.00 -> 26.3 mm
