File: Демо борд переходник/Демо итог/com_1300.kicad_pcb (KiCad board)
At the start: 4 copper layers, 50.1 x 53.2 mm, 18 parts, among them IC1 SN74CBTD3384CDBR, IC2 SN74CBTD3384CDBR, IC3 SN74CBTD3384CDBR, IC4 SN74CBTD3384CDBR, J1 9-68RD-0.635SF, J3 Conn_02x32_Top_Bottom

Commit message: 32244
Parts:
- IC4: footprint LIB_SN74CBTD3384CDBR:SOP65P780X200-24N -> SN74CBTD3384CDBR:SOP65P780X200-24N
Connections:
- J1 pad 18: VCC -> unconnected-(J1-VPP1-Pad18)
- J1 pad 42: unconnected-(J1-CE2#-Pad42) -> CE2#
- J1 pad 43: unconnected-(J1-VS1#/Refresh-Pad43) -> VS1/REFRESH
- J1 pad 52: VCC -> unconnected-(J1-VPP2-Pad52)
- J3 pad 30: unconnected-(J3-Pin_30-Pad30) -> VS1/REFRESH
- J3 pad 31: unconnected-(J3-Pin_31-Pad31) -> RESET
- J3 pad 62: unconnected-(J3-Pin_62-Pad62) -> CE2#
Routing:
- net VS1/REFRESH: track 0.00 -> 103.7 mm, vias 0 -> 2
- net CE2#: track 0.00 -> 59.4 mm, vias 0 -> 2
- net RESET: track 7.81 -> 57.3 mm, vias 0 -> 1
Other:
- board size 50.1 x 53.2 mm -> 50 x 53.2 mm
- board text added: "VS1"
