File: Демо борд переходник/Демо итог/com_1300.kicad_sch (KiCad schematic)
At the start: 19 parts, among them IC1 SN74CBTD3384CDBR, IC2 SN74CBTD3384CDBR, IC3 SN74CBTD3384CDBR, IC4 SN74CBTD3384CDBR, J1 9-68RD-0.635SF, J2 Conn_02x32_Top_Bottom, J3 Conn_02x32_Top_Bottom

Commit message: 32244
Connections:
- net RESET: now also J3.31 (Pin_31)
- net VCC: no longer J1.18 (VPP1), J1.52 (VPP2)
- net VS1/REFRESH: now reaches J3.30 (Pin_30)
- net VS1/REFRESH: now also J1.43 (VS1#/Refresh)
- net CE2#: now reaches J3.62 (Pin_62)
- net CE2#: now also J1.42 (CE2#)
- no-connect marks 56 -> 49
Other:
- moved on the sheet: C1, C2, C3, C4, IC1, IC2, IC3, IC4, J2, J3, R2
